File: Computer Designs/Cykomputer/vgacard.kicad_sch (KiCad schematic)
At the start: 0 parts

Commit message: Continued
Changed lines of the file:
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@@
 	(paper "A4")
 	(hierarchical_label "H3"
-		(shape input)
-		(at 201.93 54.61 0)
+		(shape output)
+		(at 234.95 58.42 0)
 		(effects
 			(font
@@
 	)
 	(hierarchical_label "H1"
-		(shape input)
-		(at 201.93 49.53 0)
-		(effects
-			(font
-				(size 1.27 1.27)
-			)
-			(justify left)
+		(shape output)
+		(at 234.95 53.34 0)
+		(effects
+			(font
+				(size 1.27 1.27)
+			)
+			(justify left)
+		)
+	)
+	(hierarchical_label "R"
+		(shape output)
+		(at 127 49.53 180)
+		(effects
+			(font
+				(size 1.27 1.27)
+			)
+			(justify right)
 		)
 	)
 	(hierarchical_label "V0"
-		(shape input)
-		(at 201.93 67.31 0)
+		(shape output)
+		(at 234.95 76.2 0)
 		(effects
 			(font
@@
 	)
 	(hierarchical_label "H5"
-		(shape input)
-		(at 201.93 59.69 0)
-		(effects
-			(font
-				(size 1.27 1.27)
-			)
-			(justify left)
+		(shape output)
+		(at 234.95 63.5 0)
+		(effects
+			(font
+				(size 1.27 1.27)
+			)
+			(justify left)
+		)
+	)
+	(hierarchical_label "VBLANK"
+		(shape output)
+		(at 127 64.77 180)
+		(effects
+			(font
+				(size 1.27 1.27)
+			)
+			(justify right)
 		)
 	)
 	(hierarchical_label "H6"
-		(shape input)
-		(at 201.93 62.23 0)
-		(effects
-			(font
-				(size 1.27 1.27)
-			)
-			(justify left)
+		(shape output)
+		(at 234.95 66.04 0)
+		(effects
+			(font
+				(size 1.27 1.27)
+			)
+			(justify left)
+		)
+	)
+	(hierarchical_label "HBLANK"
+		(shape output)
+		(at 127 59.69 180)
+		(effects
+			(font
+				(size 1.27 1.27)
+			)
+			(justify right)
 		)
 	)
 	(hierarchical_label "H4"
-		(shape input)
-		(at 201.93 57.15 0)
+		(shape output)
+		(at 234.95 60.96 0)
 		(effects
 			(font
@@
 	)
 	(hierarchical_label "V7"
-		(shape input)
-		(at 201.93 85.09 0)
+		(shape output)
+		(at 234.95 93.98 0)
+		(effects
+			(font
+				(size 1.27 1.27)
+			)
+			(justify left)
+		)
+	)
+	(hierarchical_label "D3"
+		(shape input)
+		(at 234.95 109.22 0)
 		(effects
 			(font
@@
 	)
 	(hierarchical_label "H7"
-		(shape input)
-		(at 201.93 64.77 0)
+		(shape output)
+		(at 234.95 68.58 0)
 		(effects
 			(font
@@
 	)
 	(hierarchical_label "V6"
-		(shape input)
-		(at 201.93 82.55 0)
+		(shape output)
+		(at 234.95 91.44 0)
+		(effects
+			(font
+				(size 1.27 1.27)
+			)
+			(justify left)
+		)
+	)
+	(hierarchical_label "HSYNC"
+		(shape output)
+		(at 127 57.15 180)
+		(effects
+			(font
+				(size 1.27 1.27)
+			)
+			(justify right)
+		)
+	)
+	(hierarchical_label "VCC"
+		(shape bidirectional)
+		(at 234.95 25.4 0)
 		(effects
 			(font
@@
 	)
 	(hierarchical_label "V5"
-		(shape input)
-		(at 201.93 80.01 0)
+		(shape output)
+		(at 234.95 88.9 0)
+		(effects
+			(font
+				(size 1.27 1.27)
+			)
+			(justify left)
+		)
+	)
+	(hierarchical_label "B"
+		(shape output)
+		(at 127 54.61 180)
+		(effects
+			(font
+				(size 1.27 1.27)
+			)
+			(justify right)
+		)
+	)
+	(hierarchical_label "G"
+		(shape output)
+		(at 127 52.07 180)
+		(effects
+			(font
+				(size 1.27 1.27)
+			)
+			(justify right)
+		)
+	)
+	(hierarchical_label "D0"
+		(shape input)
+		(at 234.95 101.6 0)
+		(effects
+			(font
+				(size 1.27 1.27)
+			)
+			(justify left)
+		)
+	)
+	(hierarchical_label "VSYNC"
+		(shape output)
+		(at 127 62.23 180)
+		(effects
+			(font
+				(size 1.27 1.27)
+			)
+			(justify right)
+		)
+	)
+	(hierarchical_label "D7"
+		(shape input)
+		(at 234.95 119.38 0)
+		(effects
+			(font
+				(size 1.27 1.27)
+			)
+			(justify left)
+		)
+	)
+	(hierarchical_label "D1"
+		(shape input)
+		(at 234.95 104.14 0)
 		(effects
 			(font
@@
 	)
 	(hierarchical_label "V2"
-		(shape input)
-		(at 201.93 72.39 0)
+		(shape output)
+		(at 234.95 81.28 0)
 		(effects
 			(font
@@
 	)
 	(hierarchical_label "V3"
-		(shape input)
-		(at 201.93 74.93 0)
+		(shape output)
+		(at 234.95 83.82 0)
+		(effects
+			(font
+				(size 1.27 1.27)
+			)
+			(justify left)
+		)
+	)
+	(hierarchical_label "D5"
+		(shape input)
+		(at 234.95 114.3 0)
+		(effects
+			(font
+				(size 1.27 1.27)
+			)
+			(justify left)
+		)
+	)
+	(hierarchical_label "D2"
+		(shape input)
+		(at 234.95 106.68 0)
 		(effects
 			(font
@@
 	)
 	(hierarchical_label "H0"
-		(shape input)
-		(at 201.93 46.99 0)
+		(shape output)
+		(at 234.95 50.8 0)
+		(effects
+			(font
+				(size 1.27 1.27)
+			)
+			(justify left)
+		)
+	)
+	(hierarchical_label "D6"
+		(shape input)
+		(at 234.95 116.84 0)
+		(effects
+			(font
+				(size 1.27 1.27)
+			)
+			(justify left)
+		)
+	)
+	(hierarchical_label "D4"
+		(shape input)
+		(at 234.95 111.76 0)
 		(effects
 			(font
@@
 	)
 	(hierarchical_label "V1"
-		(shape input)
-		(at 201.93 69.85 0)
+		(shape output)
+		(at 234.95 78.74 0)
 		(effects
 			(font
@@
 	)
 	(hierarchical_label "H2"
-		(shape input)
-		(at 201.93 52.07 0)
+		(shape output)
+		(at 234.95 55.88 0)
+		(effects
+			(font
+				(size 1.27 1.27)
+			)
+			(justify left)
+		)
+	)
+	(hierarchical_label "CHIP_ENABLE"
+		(shape output)
+		(at 234.95 127 0)
+		(effects
+			(font
+				(size 1.27 1.27)
+			)
+			(justify left)
+		)
+	)
+	(hierarchical_label "GND"
+		(shape bidirectional)
+		(at 234.95 27.94 0)
 		(effects
 			(font
@@
 	)
 	(hierarchical_label "V4"
-		(shape input)
-		(at 201.93 77.47 0)
-		(effects
-			(font
+		(shape output)
+		(at 234.95 86.36 0)
+		(effects
+			(font

Commit message: Continued
Changed lines of the file:
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@@
 	(generator_version "10.0")
 	(paper "A4")
+	(label "VCC"
+		(at 234.95 25.4 180)
+		(effects
+			(font
+				(size 1.27 1.27)
+			)
+			(justify right bottom)
+		)
+	)
+	(label "GND"
+		(at 234.95 34.29 180)
+		(effects
+			(font
+				(size 1.27 1.27)
+			)
+			(justify right bottom)
+		)
+	)
 	(hierarchical_label "H3"
 		(shape output)
@@
 	(hierarchical_label "GND"
 		(shape bidirectional)
-		(at 234.95 27.94 0)
+		(at 234.95 34.29 0)
 		(effects
 			(font
@@
 		)
 	)
+	(symbol
+		(lib_id "power:PWR_FLAG")
+		(at 234.95 25.4 0)
+		(unit 1)
+		(body_style 1)
+		(exclude_from_sim no)
+		(in_bom yes)
+		(on_board yes)
+		(in_pos_files yes)
+		(dnp no)
+		(fields_autoplaced yes)
+		(property "Reference" "#FLG03"
+			(at 234.95 23.495 0)
+			(hide yes)
+			(show_name no)
+			(do_not_autoplace no)
+			(effects
+				(font
+					(size 1.27 1.27)
+				)
+			)
+		)
+		(property "Value" "PWR_FLAG"
+			(at 234.95 20.32 0)
+			(show_name no)
+			(do_not_autoplace no)
+			(effects
+				(font
+					(size 1.27 1.27)
+				)
+			)
+		)
+		(property "Footprint" ""
+			(at 234.95 25.4 0)
+			(hide yes)
+			(show_name no)
+			(do_not_autoplace no)
+			(effects
+				(font
+					(size 1.27 1.27)
+				)
+			)
+		)
+		(property "Datasheet" ""
+			(at 234.95 25.4 0)
+			(hide yes)
+			(show_name no)
+			(do_not_autoplace no)
+			(effects
+				(font
+					(size 1.27 1.27)
+				)
+			)
+		)
+		(property "Description" "Special symbol for telling ERC where power comes from"
+			(at 234.95 25.4 0)
+			(hide yes)
+			(show_name no)
+			(do_not_autoplace no)
+			(effects
+				(font
+					(size 1.27 1.27)
+				)
+			)
+		)
+		(pin "1"
+		)
+		(instances
+			(project "Cykomputer"
+				(path "/7319cfd4-b54a-49cd-84bf-92265ba5acc0/94db923e-9f09-4888-9e9d-c984b6a27067"
+					(reference "#FLG03")
+					(unit 1)
+				)
+			)
+		)
+	)
+	(symbol
+		(lib_id "power:PWR_FLAG")
+		(at 234.95 34.29 0)
+		(unit 1)
+		(body_style 1)
+		(exclude_from_sim no)
+		(in_bom yes)
+		(on_board yes)
+		(in_pos_files yes)
+		(dnp no)
+		(fields_autoplaced yes)
+		(property "Reference" "#FLG04"
+			(at 234.95 32.385 0)
+			(hide yes)
+			(show_name no)
+			(do_not_autoplace no)
+			(effects
+				(font
+					(size 1.27 1.27)
+				)
+			)
+		)
+		(property "Value" "PWR_FLAG"
+			(at 234.95 29.21 0)
+			(show_name no)
+			(do_not_autoplace no)
+			(effects
+				(font
+					(size 1.27 1.27)
+				)
+			)
+		)
+		(property "Footprint" ""
+			(at 234.95 34.29 0)
+			(hide yes)
+			(show_name no)
+			(do_not_autoplace no)
+			(effects
+				(font
+					(size 1.27 1.27)
+				)
+			)
+		)
+		(property "Datasheet" ""
+			(at 234.95 34.29 0)
+			(hide yes)
+			(show_name no)
+			(do_not_autoplace no)
+			(effects
+				(font
+					(size 1.27 1.27)
+				)
+			)
+		)
+		(property "Description" "Special symbol for telling ERC where power comes from"
+			(at 234.95 34.29 0)
+			(hide yes)
+			(show_name no)
+			(do_not_autoplace no)
+			(effects
+				(font
+					(size 1.27 1.27)
+				)
+			)
+		)
+		(pin "1"
+		)
+		(instances
+			(project "Cykomputer"
+				(path "/7319cfd4-b54a-49cd-84bf-92265ba5acc0/94db923e-9f09-4888-9e9d-c984b6a27067"
+					(reference "#FLG04")
+					(unit 1)
+				)
+			)
+		)
+	)
