File: Computer Designs/Cykomputer/Cykomputer.kicad_sch (KiCad schematic)
At the start: 64 parts, among them J1 Bus_ISA_8bit, J10 DE15_Socket_HighDensity_Mount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, J12 IEC_60320_C14_Receptacle, J13 Conn_01x02, J14 PINHD_1x2_Male, J15 Bus_ISA_8bit, J16 Conn_02x12_Row_Letter_First, J17 Conn_01x12, J2 Bus_ISA_8bit, J3 Bus_ISA_8bit, J4 DE9_Pins_MountingHoles, J5 DE9_Pins_MountingHoles, J6 Mini-DIN-6, J7 DE15_Socket_HighDensity_Mount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, J8 DE15_Socket_HighDensity_Mount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, J9 DE15_Socket_HighDensity_Mount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, P1 USB_C_Plug_USB2.0, SW1 SW_SPST, SW2 SW_Rotary_1x7_MP, U1 W65C02SxP, U10 74HC14, U12 W65C02SxP, U13 27C256, U14 KM62256CLP, U15 KM62256CLP, U16 27C256, U17 74HCT595, U18 74HCT164, U19 KM62256CLP, U2 W65C22SxP, U22 W65C22SxP, U23 74HCT595, U24 74HCT595, U25 KM62256CLP, U26 W65C22SxP, U3 W65C22SxP, U4 W65C22SxP, U5 W65C51NxP, U6 W65C51NxP, U7 MAX232, U8 MAX232, U9 W65C22SxP, Y1 ACO-xxxMHz-A, Y2 ACO-xxxMHz-A, Y3 ACO-xxxMHz-A, Y4 ACO-xxxMHz-A, Y5 ACO-xxxMHz-A, Y6 ACO-xxxMHz-A, Y7 ACO-xxxMHz-A

Commit message: Updated Computer schematic
Parts:
- removed P1: USB_C_Plug_USB2.0, symbol Connector:USB_C_Plug_USB2.0
- added C11: 100nF_Ceramic, Capacitor_THT:C_Disc_D5.0mm_W2.5mm_P2.50mm, symbol PCM_SL_Capacitors:100nF_Ceramic
- added J11: USB_C_Receptacle, symbol Connector:USB_C_Receptacle
- added U11: W65C51NxP, Package_DIP:DIP-28_W15.24mm, symbol PCM_65xx-library:W65C51NxP
- added U20: 4053, symbol 4xxx:4053
- added U21: MIC2025-2YM, Package_SO:SOIC-8_3.9x4.9mm_P1.27mm, symbol Power_Management:MIC2025-2YM
- added U27: CH340G, Package_SO:SOIC-16_3.9x9.9mm_P1.27mm, symbol Interface_USB:CH340G
Connections:
- net GND: now also C11.2, J11.A1 (GND), J11.A12 (GND), J11.B1 (GND), J11.B12 (GND), J11.SH (SHIELD), U11.1 (VSS), U20.8 (VSS), U21.3 (GND), U27.1 (GND)
- net Serial Clock: now also U11.6 (XTAL1)
- net VCC: now also U11.15 (VCC), U20.16 (VDD), U21.7 (IN), U27.16 (VCC)
- net at SW2.8, U1.39 (ϕ2), U5.27 (ϕ2)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: now also U11.4 (~{RES})
- new net: C11.1, J11.A4 (VBUS), J11.A9 (VBUS), J11.B4 (VBUS), J11.B9 (VBUS), U21.6 (OUT), U21.8 (OUT)

Commit message: Continued
Parts:
- removed C1: C, symbol Device:C
- added C1: 470uF, PCM_SparkFun-Capacitor:Electrolytic_10.3x10.3mm, symbol PCM_SparkFun-Capacitor:470uF_10x10_25V_20%
Connections:
- net VCC: now also C1.1; no longer J1.29 (VCC), J1.3 (VCC), J15.29 (VCC), J15.3 (VCC), J16.a1 (Pin_a1), J17.1 (Pin_1), J2.29 (VCC), J2.3 (VCC), J3.29 (VCC), J3.3 (VCC), J6.4, R3.2, R5.1, U1.8 (VDD), U10.14 (VCC), U12.8 (VDD), U13.28 (VCC), U14.28 (VCC), U15.28 (VCC), U17.16 (VCC), U18.14 (VCC), U2.20 (VCC), U22.20 (VCC), U23.10 (~{SRCLR}), U23.16 (VCC), U24.10 (~{SRCLR}), U24.16 (VCC), U25.28 (VCC), U26.20 (VCC), U3.20 (VCC), U4.20 (VCC), U5.15 (VCC), U7.16 (VCC), U9.20 (VCC)
- net RST: now reaches J13.2 (Pin_2), R3.1, U1.40 (~{RES}), U12.40 (~{RES}), U2.34 (~{RES}), U3.34 (~{RES}), U4.34 (~{RES}), U5.4 (~{RES}), U6.4 (~{RES})
- new net: C1.2, J1.29 (VCC), J1.3 (VCC), J15.29 (VCC), J15.3 (VCC), J16.a1 (Pin_a1), J17.1 (Pin_1), J2.29 (VCC), J2.3 (VCC), J3.29 (VCC), J3.3 (VCC), J6.4, R3.2, R5.1, U1.8 (VDD), U10.14 (VCC), U12.8 (VDD), U13.28 (VCC), U14.28 (VCC), U15.28 (VCC), U17.16 (VCC), U18.14 (VCC), U2.20 (VCC), U22.20 (VCC), U23.10 (~{SRCLR}), U23.16 (VCC), U24.10 (~{SRCLR}), U24.16 (VCC), U25.28 (VCC), U26.20 (VCC), U3.20 (VCC), U4.20 (VCC), U5.15 (VCC), U7.16 (VCC), U9.20 (VCC)
Changed lines of the file:
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@@
 	)
 	(junction
-		(at 588.01 205.74)
-		(diameter 0)
-		(color 0 0 0 0)
-	)
-	(junction
 		(at 96.52 205.74)
 		(diameter 0)
@@
 	)
 	(junction
-		(at 580.39 205.74)
-		(diameter 0)
-		(color 0 0 0 0)
-	)
-	(junction
 		(at 452.12 210.82)
 		(diameter 0)
@@
 	(wire
 		(pts
-			(xy 588.01 201.93) (xy 588.01 205.74)
-		)
-		(stroke
-			(width 0)
-			(type default)
-			(color 255 0 0 1)
-		)
-	)
-	(wire
-		(pts
 			(xy 417.83 184.15) (xy 417.83 175.26)
 		)
@@
 	(wire
 		(pts
+			(xy 579.12 205.74) (xy 596.9 205.74)
+		)
+		(stroke
+			(width 0)
+			(type default)
+			(color 255 0 0 1)
+		)
+	)
+	(wire
+		(pts
 			(xy 434.34 101.6) (xy 443.23 101.6)
 		)
@@
 	(wire
 		(pts
-			(xy 580.39 205.74) (xy 588.01 205.74)
-		)
-		(stroke
-			(width 0)
-			(type default)
-			(color 255 0 0 1)
-		)
-	)
-	(wire
-		(pts
 			(xy 454.66 134.62) (xy 459.74 134.62)
 		)
@@
 	(wire
 		(pts
-			(xy 588.01 205.74) (xy 596.9 205.74)
-		)
-		(stroke
-			(width 0)
-			(type default)
-			(color 255 0 0 1)
-		)
-	)
-	(wire
-		(pts
 			(xy 518.16 96.52) (xy 518.16 146.05)
 		)
@@
 	(wire
 		(pts
-			(xy 557.53 205.74) (xy 580.39 205.74)
+			(xy 557.53 205.74) (xy 574.04 205.74)
 		)
 		(stroke
@@
 	(wire
 		(pts
-			(xy 580.39 201.93) (xy 580.39 205.74)
-		)
-		(stroke
-			(width 0)
-			(type default)
-			(color 255 0 0 1)
-		)
-	)
-	(wire
-		(pts
 			(xy 85.09 210.82) (xy 151.13 210.82)
 		)
@@
 		)
 	)
+	(label "RST"
+		(at 379.73 369.57 0)
+		(effects
+			(font
+				(size 1.27 1.27)
+			)
+			(justify left bottom)
+		)
+	)
 	(label "D5"
 		(at 430.53 449.58 180)
@@
 	(symbol
 		(lib_id "Device:C")
-		(at 584.2 201.93 270)
-		(unit 1)
-		(body_style 1)
-		(exclude_from_sim no)
-		(in_bom yes)
-		(on_board yes)
-		(in_pos_files yes)
-		(dnp no)
-		(fields_autoplaced yes)
-		(property "Reference" "C1"
-			(at 584.2 194.31 90)
-			(show_name no)
-			(do_not_autoplace no)
-			(effects
-				(font
-					(size 1.27 1.27)
-				)
-			)
-		)
-		(property "Value" "C"
-			(at 584.2 196.85 90)
-			(show_name no)
-			(do_not_autoplace no)
-			(effects
-				(font
-					(size 1.27 1.27)
-				)
-			)
-		)
-		(property "Footprint" ""
-			(at 580.39 202.8952 0)
-			(hide yes)
-			(show_name no)
-			(do_not_autoplace no)
-			(effects
-				(font
-					(size 1.27 1.27)
-				)
-			)
-		)
-		(property "Datasheet" ""
-			(at 584.2 201.93 0)
-			(hide yes)
-			(show_name no)
-			(do_not_autoplace no)
-			(effects
-				(font
-					(size 1.27 1.27)
-				)
-			)
-		)
-		(property "Description" "Unpolarized capacitor"
-			(at 584.2 201.93 0)
-			(hide yes)
-			(show_name no)
-			(do_not_autoplace no)
-			(effects
-				(font
-					(size 1.27 1.27)
-				)
-			)
-		)
-		(pin "1"
-		)
-		(pin "2"
-		)
-		(instances
-			(project "Cykomputer"
-				(path "/7319cfd4-b54a-49cd-84bf-92265ba5acc0"
-					(reference "C1")
-					(unit 1)
-				)
-			)
-		)
-	)
-	(symbol
-		(lib_id "Device:C")
 		(at 669.29 373.38 0)
 		(unit 1)
@@
 	)
 	(symbol
+		(lib_id "PCM_SparkFun-Capacitor:470uF_10x10_25V_20%")
+		(at 576.58 205.74 270)
+		(unit 1)
+		(body_style 1)
+		(exclude_from_sim no)
+		(in_bom yes)
+		(on_board yes)
+		(in_pos_files yes)
+		(dnp no)
+		(fields_autoplaced yes)
+		(property "Reference" "C1"
+			(at 577.0118 194.31 90)
+			(show_name no)
+			(do_not_autoplace no)
+			(effects
+				(font
+					(size 1.27 1.27)
+				)
+			)
+		)
+		(property "Value" "470uF"
+			(at 577.0118 196.85 90)
+			(show_name no)
+			(do_not_autoplace no)
+			(effects
+				(font
+					(size 1.27 1.27)
+				)
+			)
+		)
+		(property "Footprint" "PCM_SparkFun-Capacitor:Electrolytic_10.3x10.3mm"
+			(at 558.8 205.74 0)
+			(hide yes)
+			(show_name no)
+			(do_not_autoplace no)
+			(effects
+				(font
+					(size 1.27 1.27)
+				)
+			)
+		)
+		(property "Datasheet" "https://www.nichicon.co.jp/english/series_items/catalog_pdf/e-uud.pdf"
+			(at 561.34 207.01 0)
+			(hide yes)
+			(show_name no)
+			(do_not_autoplace no)
+			(effects
+				(font
+					(size 1.27 1.27)
+				)
+			)
+		)
+		(property "Description" "Polarized capacitor, US symbol"
+			(at 556.26 205.74 0)
+			(hide yes)
+			(show_name no)
+			(do_not_autoplace no)
+			(effects
+				(font
+					(size 1.27 1.27)
+				)
+			)
+		)
+		(property "PROD_ID" ""
+			(at 563.88 205.74 0)
+			(hide yes)
+			(show_name no)
+			(do_not_autoplace no)
+			(effects
+				(font
+					(size 1.27 1.27)
+				)
+			)
+		)
+		(property "Voltage" "25V"
+			(at 577.0118 199.39 90)
+			(show_name no)
+			(do_not_autoplace no)
+			(effects
+				(font
+					(size 1.27 1.27)
+				)
+			)
+		)
+		(property "Tolerance" "20%"
+			(at 577.0118 201.93 90)
+			(show_name no)
+			(do_not_autoplace no)
+			(effects
+				(font
+					(size 1.27 1.27)
+				)
+			)
+		)
+		(pin "2"
+		)
+		(pin "1"
+		)
+		(instances
+			(project "Cykomputer"
+				(path "/7319cfd4-b54a-49cd-84bf-92265ba5acc0"
+					(reference "C1")
+					(unit 1)
+				)
+			)
+		)
+	)
+	(symbol
 		(lib_id "Device:C")
 		(at 119.38 389.89 90)
@@
 			)
 		)
-		(pin "H0" input
+		(pin "H0" output
 			(at 359.41 36.83 0)
 			(effects
@@
 			)
 		)
-		(pin "H1" input
+		(pin "H1" output
 			(at 359.41 38.1 0)
 			(effects
@@
 			)
 		)
-		(pin "H2" input
+		(pin "H2" output
 			(at 359.41 39.37 0)
 			(effects
@@
 			)
 		)
-		(pin "H3" input
+		(pin "H3" output
 			(at 359.41 40.64 0)
 			(effects
@@
 			)
 		)
-		(pin "H4" input
+		(pin "H4" output
 			(at 359.41 41.91 0)
 			(effects
@@
 			)
 		)
-		(pin "H5" input
+		(pin "H5" output
 			(at 359.41 43.18 0)
 			(effects
@@
 			)
 		)
-		(pin "H6" input
+		(pin "H6" output
 			(at 359.41 44.45 0)
 			(effects
@@
 			)
 		)
-		(pin "H7" input
+		(pin "H7" output
 			(at 359.41 45.72 0)
 			(effects
@@
 			)
 		)
-		(pin "V0" input
+		(pin "V0" output
 			(at 359.41 46.99 0)
 			(effects
@@
 			)
 		)
-		(pin "V1" input
+		(pin "V1" output
 			(at 359.41 48.26 0)
 			(effects
@@
 			)
 		)
-		(pin "V2" input
+		(pin "V2" output
 			(at 359.41 49.53 0)
 			(effects
@@
 			)
 		)
-		(pin "V3" input
+		(pin "V3" output
 			(at 359.41 50.8 0)
 			(effects
@@
 			)
 		)
-		(pin "V4" input
+		(pin "V4" output
 			(at 359.41 52.07 0)
 			(effects
@@
 			)
 		)
-		(pin "V5" input
+		(pin "V5" output
 			(at 359.41 53.34 0)
 			(effects
@@
 			)
 		)
-		(pin "V6" input
+		(pin "V6" output
 			(at 359.41 54.61 0)
 			(effects
@@
 			)
 		)
-		(pin "V7" input
+		(pin "V7" output
 			(at 359.41 55.88 0)
 			(effects

Commit message: Continued
Parts:
- added U28: LM809, Package_TO_SOT_SMD:SOT-23, symbol Power_Supervisor:LM809
Connections:
- net GND: now also U28.1 (GND)
- net RST: now also U28.2 (~{RESET})
- net at C1.2, J1.29 (VCC), J1.3 (VCC)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: now also U28.3 (VCC)
Changed lines of the file:
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@@
 	)
 	(junction
+		(at 360.68 389.89)
+		(diameter 0)
+		(color 0 0 0 0)
+	)
+	(junction
 		(at 123.19 389.89)
 		(diameter 0)
@@
 	)
 	(junction
+		(at 353.06 379.73)
+		(diameter 0)
+		(color 0 0 0 0)
+	)
+	(junction
 		(at 280.67 139.7)
 		(diameter 0)
@@
 	)
 	(junction
+		(at 335.28 400.05)
+		(diameter 0)
+		(color 0 0 0 0)
+	)
+	(junction
 		(at 455.93 189.23)
 		(diameter 0)
@@
 	(wire
 		(pts
+			(xy 335.28 400.05) (xy 350.52 400.05)
+		)
+		(stroke
+			(width 0)
+			(type default)
+			(color 0 0 0 1)
+		)
+	)
+	(wire
+		(pts
 			(xy 490.22 246.38) (xy 443.23 246.38)
 		)
@@
 	(wire
 		(pts
-			(xy 335.28 464.82) (xy 335.28 381)
+			(xy 335.28 464.82) (xy 335.28 400.05)
 		)
 		(stroke
@@
 	(wire
 		(pts
+			(xy 353.06 379.73) (xy 353.06 381)
+		)
+		(stroke
+			(width 0)
+			(type default)
+			(color 255 0 0 1)
+		)
+	)
+	(wire
+		(pts
 			(xy 372.11 349.25) (xy 372.11 354.33)
 		)
@@
 	(wire
 		(pts
+			(xy 335.28 400.05) (xy 335.28 381)
+		)
+		(stroke
+			(width 0)
+			(type default)
+			(color 0 0 0 1)
+		)
+	)
+	(wire
+		(pts
 			(xy 520.7 140.97) (xy 520.7 91.44)
 		)
@@
 	(wire
 		(pts
+			(xy 358.14 389.89) (xy 360.68 389.89)
+		)
+		(stroke
+			(width 0)
+			(type default)
+		)
+	)
+	(wire
+		(pts
 			(xy 455.93 189.23) (xy 459.74 189.23)
 		)
@@
 	(wire
 		(pts
-			(xy 353.06 347.98) (xy 353.06 381)
+			(xy 353.06 347.98) (xy 353.06 379.73)
 		)
 		(stroke
@@
 	(wire
 		(pts
+			(xy 350.52 379.73) (xy 353.06 379.73)
+		)
+		(stroke
+			(width 0)
+			(type default)
+			(color 255 0 0 1)
+		)
+	)
+	(wire
+		(pts
 			(xy 462.28 279.4) (xy 462.28 278.13)
 		)
@@
 					(unit 1)
 				)
+			)
+		)
+	)
+	(symbol
+		(lib_id "Power_Supervisor:LM809")
+		(at 350.52 389.89 0)
+		(unit 1)
+		(body_style 1)
+		(exclude_from_sim no)
+		(in_bom yes)
+		(on_board yes)
+		(in_pos_files yes)
+		(dnp no)
+		(fields_autoplaced yes)
+		(property "Reference" "U28"
+			(at 344.17 388.6199 0)
+			(show_name no)
+			(do_not_autoplace no)
+			(effects
+				(font
+					(size 1.27 1.27)
+				)
+				(justify right)
+			)
+		)
+		(property "Value" "LM809"
+			(at 344.17 391.1599 0)
+			(show_name no)
+			(do_not_autoplace no)
+			(effects
+				(font
+					(size 1.27 1.27)
+				)
+				(justify right)
+			)
+		)
+		(property "Footprint" "Package_TO_SOT_SMD:SOT-23"
+			(at 358.14 387.35 0)
+			(hide yes)
+			(show_name no)
+			(do_not_autoplace no)
+			(effects
+				(font
+					(size 1.27 1.27)
+				)
+			)
+		)
+		(property "Datasheet" "http://www.ti.com/lit/ds/symlink/lm809.pdf"
+			(at 358.14 387.35 0)
+			(hide yes)
+			(show_name no)
+			(do_not_autoplace no)
+			(effects
+				(font
+					(size 1.27 1.27)
+				)
+			)
+		)
+		(property "Description" "Microprocessor Reset (active-low) Circuit, SOT-23"
+			(at 350.52 389.89 0)
+			(hide yes)
+			(show_name no)
+			(do_not_autoplace no)
+			(effects
+				(font
+					(size 1.27 1.27)
+				)
+			)
+		)
+		(pin "1"
+		)
+		(pin "2"
+		)
+		(pin "3"
+		)
+		(instances
+			(project "Cykomputer"
+				(path "/7319cfd4-b54a-49cd-84bf-92265ba5acc0"
+					(reference "U28")
+					(unit 1)
+				)

Commit message: Continued
Parts:
- removed U28: LM809, Package_TO_SOT_SMD:SOT-23, symbol Power_Supervisor:LM809
- added U28: DS1813-5, Package_TO_SOT_THT:TO-92, symbol Cykomputer-Parts:DS1813-5
- added U29: CH376S, Package_SO:SOIC-28W_7.5x17.9mm_P1.27mm, symbol Cykomputer-Parts:CH376S
Connections:
- net GND: now also U28.3 (GND), U29.12 (GND)
- net RST: now also U28.1 (~{RESET})
- net VCC: now also U29.28 (VCC)
- net at C1.2, J1.29 (VCC), J1.3 (VCC)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: now also U28.2 (VCC)
- net VIDEO_BIT0: now reaches U26.2 (PA0)
- net VIDEO_BIT0: now also U22.2 (PA0)
- net VIDEO_BIT1: now reaches U26.3 (PA1)
- net VIDEO_BIT1: now also U22.3 (PA1)
- net VIDEO_BIT2: now reaches U26.4 (PA2)
- net VIDEO_BIT2: now also U22.4 (PA2)
- net VIDEO_BIT3: now reaches U26.5 (PA3)
- net VIDEO_BIT3: now also U22.5 (PA3)
- net VIDEO_BIT4: now reaches U26.6 (PA4)
- net VIDEO_BIT4: now also U22.6 (PA4)
- net VIDEO_BIT5: now reaches U26.7 (PA5)
- net VIDEO_BIT5: now also U22.7 (PA5)
- net VIDEO_BIT6: now reaches U26.8 (PA6)
- net VIDEO_BIT6: now also U22.8 (PA6)
- net VIDEO_BIT7: now reaches U26.9 (PA7)
- net VIDEO_BIT7: now also U22.9 (PA7)
Other:
- sheet VGA Controller ports: added B, CHIP_ENABLE, D0, D1, D2, D3, D4, D5, D6, D7, G, GND, HBLANK, HSYNC, R, VBLANK, VCC, VSYNC; removed none
- note added: "1000 Available Addresses"
- note added: "Banking & Timers & Video"
- note added: "Video Data Input & Banking"
- note removed: "Banking & Timers"

Commit message: Continued
Parts:
- removed U2, U3: W65C22SxP, Package_DIP:DIP-40_W15.24mm, symbol PCM_65xx-library:W65C22SxP
- added 5V 5A Wall AC/DC Adapter2: (no value), symbol Cykomputer-Parts:Power-Supply-5V-5A
- added J18: AudioJack2, symbol Connector_Audio:AudioJack2
- added J19: Conn_01x32, symbol Connector_Generic:Conn_01x32
- added J20: Conn_01x09, 4ms_Connector:Pins_1x09_2.54mm_TH, symbol PCM_4ms_Connector:Conn_01x09
- added R1: 3.3k, Resistor_THT:R_Axial_DIN0207_L6.3mm_D2.5mm_P10.16mm_Horizontal, symbol PCM_SL_Resistors:3.3k
- added SW3: Push_Button, Button_Switch_THT:SW_PUSH_6mm, symbol PCM_SL_Devices:Push_Button
- added U30: 6581, Package_DIP:DIP-28_W15.24mm, symbol PCM_65xx-library:6581
Connections:
- net D0: now also J19.32 (Pin_32), U30.15 (D0)
- net D1: now also J19.31 (Pin_31), U30.16 (D1)
- net D2: now also J19.30 (Pin_30), U30.17 (D2)
- net D3: now also J19.29 (Pin_29), U30.18 (D3)
- net D4: now also J19.28 (Pin_28), U30.19 (D4)
- net D5: now also J19.27 (Pin_27), U30.20 (D5)
- net D6: now also J19.26 (Pin_26), U30.21 (D6)
- net D7: now also J19.25 (Pin_25), U30.22 (D7)
- net GND: now also 5V 5A Wall AC/DC Adapter2.4 (GND), J18.T, U30.14 (GND)
- net RST: now also R1.2
- net VCC: now also 5V 5A Wall AC/DC Adapter2.3 (+V)
- net at C1.2, J1.29 (VCC), J1.3 (VCC)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: now also R1.1, U30.25 (+5V)
- net at U24.1 (QB), U4.10 (PB0): now also J20.1 (Pin_1)
- net at U24.15 (QA), U4.11 (PB1): now also J20.2 (Pin_2)
- net at U23.7 (QH), U4.12 (PB2): now also J20.3 (Pin_3)
- net at U23.6 (QG), U4.13 (PB3): now also J20.4 (Pin_4)
- net at U23.5 (QF), U4.14 (PB4): now also J20.5 (Pin_5)
- net at U23.4 (QE), U4.15 (PB5): now also J20.6 (Pin_6)
- net at U23.3 (QD), U4.16 (PB6): now also J20.7 (Pin_7)
- net at U23.2 (QC), U4.17 (PB7): now also J20.8 (Pin_8)
- net at U4.18 (CB1): now also U10.4, U23.12 (RCLK), U24.12 (RCLK)
- net at U4.40 (CA1): now also J17.2 (Pin_2)
- net A15: now reaches J15.47 (BA15)
- net A15: now also J1.47 (BA15), J2.47 (BA15), J3.47 (BA15), U1.25 (A15), J19.9 (Pin_9)
- net A14: now reaches J15.48 (BA14)
- net A14: now also J1.48 (BA14), J2.48 (BA14), J3.48 (BA14), U1.24 (A14), J19.10 (Pin_10)
- net A13: now reaches J15.49 (BA13)
- net A13: now also J1.49 (BA13), J2.49 (BA13), J3.49 (BA13), U1.23 (A13), J19.11 (Pin_11)
- net A12: now reaches J15.50 (BA12)
- net A12: now also J1.50 (BA12), J2.50 (BA12), J3.50 (BA12), U1.22 (A12), J19.12 (Pin_12)
- net A11: now reaches J15.51 (BA11)
- net A11: now also J1.51 (BA11), J2.51 (BA11), J3.51 (BA11), U1.20 (A11), J19.13 (Pin_13)
- net A10: now reaches J15.52 (BA10)
- net A10: now also J1.52 (BA10), J2.52 (BA10), J3.52 (BA10), U1.19 (A10), J19.14 (Pin_14)
- net A9: now reaches J15.53 (BA09)
- net A9: now also J1.53 (BA09), J2.53 (BA09), J3.53 (BA09), U1.18 (A9), J19.15 (Pin_15)
- net A8: now reaches J15.54 (BA08)
- net A8: now also J1.54 (BA08), J2.54 (BA08), J3.54 (BA08), U1.17 (A8), J19.16 (Pin_16)
- net A7: now reaches J15.55 (BA07)
- net A7: now also J1.55 (BA07), J2.55 (BA07), J3.55 (BA07), U1.16 (A7), J19.17 (Pin_17)
- net A6: now reaches J15.56 (BA06)
- net A6: now also J1.56 (BA06), J2.56 (BA06), J3.56 (BA06), U1.15 (A6), J19.18 (Pin_18)
- net A5: now reaches J15.57 (BA05)
- net A5: now also J1.57 (BA05), J2.57 (BA05), J3.57 (BA05), U1.14 (A5), J19.19 (Pin_19)
- net A4: now reaches J15.58 (BA04)
- net A4: now also J1.58 (BA04), J2.58 (BA04), J3.58 (BA04), U1.13 (A4), J19.20 (Pin_20)
- net A3: now reaches J15.59 (BA03)
- net A3: now also J1.59 (BA03), J2.59 (BA03), J3.59 (BA03), U1.12 (A3), J19.21 (Pin_21)
- net A2: now reaches J15.60 (BA02)
- net A2: now also J1.60 (BA02), J2.60 (BA02), J3.60 (BA02), U1.11 (A2), J19.22 (Pin_22)
- net A1: now reaches J15.61 (BA01)
- net A1: now also J1.61 (BA01), J2.61 (BA01), J3.61 (BA01), U1.10 (A1), J19.23 (Pin_23)
- net A0: now reaches J15.62 (BA00)
- net A0: now also J1.62 (BA00), J2.62 (BA00), J3.62 (BA00), U1.9 (A0), J19.24 (Pin_24)
- net at J11.A6 (D+): now also J11.B6 (D+)
- net at J11.A7 (D-): now also J11.B7 (D-)
- net READ/WRITE: now reaches U1.34 (R/~{W})
- net READ/WRITE: now also J19.7 (Pin_7)
- net PHI2: now reaches SW2.8, U1.39 (ϕ2), U11.4 (~{RES}), U5.27 (ϕ2), U6.27 (ϕ2)
- net PHI2: now also J19.8 (Pin_8)
- net at 5V 5A Wall AC/DC Adapter1.1 (AC/L), SW1.2 (B): now also 5V 5A Wall AC/DC Adapter2.2 (AC/N)
- net at 5V 5A Wall AC/DC Adapter1.2 (AC/N), J12.2 (N): now also 5V 5A Wall AC/DC Adapter2.1 (AC/L)
- new net: J18.S, U30.27 (AUDIO_OUT)
- now unconnected: U16.27 (A14), U19.1 (A14), U22.10 (PB0)
- no-connect marks 44 -> 45
Other:
- note added: "$B000-$B00F"
- note added: "$B010-$B01F"
- note added: "$B020-$B02F"
- note added: "$B030-$B04F"
- note added: "$B050-$B053"
- note added: "$B054-$BO57"
- note added: "$B058-$B05B"
- note added: "$B05C-$B444"
- note added: "$B445-$B82D"
- note added: "$B82E-$BC16"
- note added: "$BC17-$BFFF"
- note added: "Function Keys"
- note added: "Sound Chip"
- note removed: "1000 Available Addresses"
- note removed: "ES2 & ES3"
- note removed: "PCI and ES1"
