File: Computer Designs/Cykomputer/Cykomputer.kicad_sch (KiCad schematic)
At the start: 78 parts, among them J1 Bus_ISA_8bit, J10 DE15_Socket_HighDensity_Mount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, J11 USB_C_Receptacle, J12 IEC_60320_C14_Receptacle, J13 Conn_01x02, J14 PINHD_1x2_Male, J15 Bus_ISA_8bit, J16 Conn_02x12_Row_Letter_First, J17 Conn_01x12, J18 AudioJack2, J19 Conn_01x32, J2 Bus_ISA_8bit, J20 Conn_01x09, J3 Bus_ISA_8bit, J4 DE9_Pins_MountingHoles, J5 DE9_Pins_MountingHoles, J6 Mini-DIN-6, J7 DE15_Socket_HighDensity_Mount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, J8 DE15_Socket_HighDensity_Mount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, J9 DE15_Socket_HighDensity_Mount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, SW1 SW_SPST, SW2 SW_Rotary_1x7_MP, SW3 Push_Button, U1 W65C02SxP, U10 74HC14, U11 W65C51NxP, U12 W65C02SxP, U13 27C256, U14 KM62256CLP, U15 KM62256CLP, U16 27C256, U17 74HCT595, U18 74HCT164, U19 KM62256CLP, U2 74LS30, U20 4053, U21 MIC2025-2YM, U22 W65C22SxP, U23 74HCT595, U24 74HCT595, U25 KM62256CLP, U26 W65C22SxP, U28 DS1813-5, U29 CH376S, U30 6581, U4 W65C22SxP, U5 W65C51NxP, U6 W65C51NxP, U7 MAX232, U8 MAX232, U9 W65C22SxP, Y1 ACO-xxxMHz-A, Y2 ACO-xxxMHz-A, Y3 ACO-xxxMHz-A, Y4 ACO-xxxMHz-A, Y5 ACO-xxxMHz-A, Y6 ACO-xxxMHz-A, Y7 ACO-xxxMHz-A

Commit message: Continued
Parts:
- added J21: Barrel_Jack_PTH, PCM_SparkFun-Connector:Barrel_Jack_PTH, symbol PCM_SparkFun-Connector:Barrel_Jack_PTH
- added J22: Conn_Receptacle_3P_Protected, PCM_SparkFun-Connector:Barrel_Jack_PTH, symbol Connector:Conn_Receptacle_3P_Protected
Connections:
- net GND: now also J21.2 (GND), J21.3 (GNDBREAK)
- net at 5V 5A Wall AC/DC Adapter1.2 (AC/N), J12.2 (N): now also 5V 5A Wall AC/DC Adapter2.2 (AC/N), J22.1 (N); no longer 5V 5A Wall AC/DC Adapter2.1 (AC/L)
- net at 5V 5A Wall AC/DC Adapter1.1 (AC/L), SW1.2 (B): now also 5V 5A Wall AC/DC Adapter2.1 (AC/L), J22.2 (L); no longer 5V 5A Wall AC/DC Adapter2.2 (AC/N)
- net 12v: now reaches J15.9 (+12V)
- net 12v: now also J1.9 (+12V), J2.9 (+12V), J3.9 (+12V), U30.28 (+12V), J21.1 (PWR)
- net at J12.3 (PE): now also J22.3 (PE)
- no-connect marks 44 -> 43
Other:
- note added: "+12v"

Commit message: Continued
Connections:
- net at U9.2 (PA0): now also J16.a6 (Pin_a6)
- net at U9.3 (PA1): now also J16.a5 (Pin_a5)
- net at U9.4 (PA2): now also J16.a4 (Pin_a4)
- net at U9.5 (PA3): now also J16.a3 (Pin_a3)
- net at U9.6 (PA4): now also J16.a2 (Pin_a2)
Changed lines of the file:
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@@
 	(wire
 		(pts
+			(xy 222.25 27.94) (xy 222.25 101.6)
+		)
+		(stroke
+			(width 0)
+			(type default)
+		)
+	)
+	(wire
+		(pts
 			(xy 509.27 148.59) (xy 516.89 148.59)
 		)
@@
 	(wire
 		(pts
+			(xy 217.17 97.79) (xy 279.4 97.79)
+		)
+		(stroke
+			(width 0)
+			(type default)
+		)
+	)
+	(wire
+		(pts
 			(xy 509.27 140.97) (xy 520.7 140.97)
 		)
@@
 	(wire
 		(pts
+			(xy 285.75 101.6) (xy 222.25 101.6)
+		)
+		(stroke
+			(width 0)
+			(type default)
+		)
+	)
+	(wire
+		(pts
 			(xy 444.5 177.8) (xy 443.23 177.8)
 		)
@@
 	(wire
 		(pts
+			(xy 217.17 27.94) (xy 217.17 97.79)
+		)
+		(stroke
+			(width 0)
+			(type default)
+		)
+	)
+	(wire
+		(pts
 			(xy 370.84 134.62) (xy 386.08 134.62)
 		)
@@
 	(wire
 		(pts
+			(xy 279.4 96.52) (xy 285.75 96.52)
+		)
+		(stroke
+			(width 0)
+			(type default)
+		)
+	)
+	(wire
+		(pts
 			(xy 426.72 279.4) (xy 427.99 279.4)
 		)
@@
 	(wire
 		(pts
+			(xy 224.79 104.14) (xy 224.79 27.94)
+		)
+		(stroke
+			(width 0)
+			(type default)
+		)
+	)
+	(wire
+		(pts
 			(xy 520.7 140.97) (xy 520.7 91.44)
 		)
@@
 	(wire
 		(pts
+			(xy 214.63 27.94) (xy 214.63 93.98)
+		)
+		(stroke
+			(width 0)
+			(type default)
+		)
+	)
+	(wire
+		(pts
 			(xy 406.4 177.8) (xy 416.56 177.8)
 		)
@@
 	(wire
 		(pts
+			(xy 219.71 99.06) (xy 285.75 99.06)
+		)
+		(stroke
+			(width 0)
+			(type default)
+		)
+	)
+	(wire
+		(pts
 			(xy 580.39 45.72) (xy 551.18 45.72)
 		)
@@
 	(wire
 		(pts
+			(xy 279.4 97.79) (xy 279.4 96.52)
+		)
+		(stroke
+			(width 0)
+			(type default)
+		)
+	)
+	(wire
+		(pts
 			(xy 415.29 311.15) (xy 426.72 311.15)
 		)
@@
 	(wire
 		(pts
+			(xy 285.75 104.14) (xy 224.79 104.14)
+		)
+		(stroke
+			(width 0)
+			(type default)
+		)
+	)
+	(wire
+		(pts
 			(xy 270.51 205.74) (xy 270.51 193.04)
 		)
@@
 	(wire
 		(pts
+			(xy 214.63 93.98) (xy 285.75 93.98)
+		)
+		(stroke
+			(width 0)
+			(type default)
+		)
+	)
+	(wire
+		(pts
 			(xy 615.95 201.93) (xy 624.84 201.93)
 		)
@@
 		)
 	)
+	(wire
+		(pts
+			(xy 219.71 27.94) (xy 219.71 99.06)
+		)
+		(stroke
+			(width 0)
+			(type default)
+		)
+	)

Commit message: Continued
Connections:
- net Variable Clock Module/CLK: now reaches SW2.7
Other:
- added sheet Variable Clock Module (clock.kicad_sch)
Changed lines of the file:
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@@
 	)
 	(junction
+		(at 600.71 339.09)
+		(diameter 0)
+		(color 0 0 0 0)
+	)
+	(junction
 		(at 212.09 68.58)
 		(diameter 0)
@@
 	)
 	(junction
+		(at 600.71 332.74)
+		(diameter 0)
+		(color 0 0 0 0)
+	)
+	(junction
 		(at 464.82 182.88)
 		(diameter 0)
@@
 	(wire
 		(pts
+			(xy 546.1 294.64) (xy 546.1 297.18)
+		)
+		(stroke
+			(width 0)
+			(type default)
+		)
+	)
+	(wire
+		(pts
 			(xy 476.25 284.48) (xy 476.25 275.59)
 		)
@@
 	(wire
 		(pts
+			(xy 541.02 321.31) (xy 541.02 297.18)
+		)
+		(stroke
+			(width 0)
+			(type default)
+		)
+	)
+	(wire
+		(pts
 			(xy 684.53 274.32) (xy 683.26 274.32)
 		)
@@
 	(wire
 		(pts
+			(xy 600.71 332.74) (xy 575.31 332.74)
+		)
+		(stroke
+			(width 0)
+			(type default)
+			(color 255 0 0 1)
+		)
+	)
+	(wire
+		(pts
 			(xy 645.16 90.17) (xy 645.16 92.71)
 		)
@@
 	(wire
 		(pts
+			(xy 575.31 332.74) (xy 575.31 330.2)
+		)
+		(stroke
+			(width 0)
+			(type default)
+			(color 255 0 0 1)
+		)
+	)
+	(wire
+		(pts
 			(xy 478.79 313.69) (xy 471.17 313.69)
 		)
@@
 	(wire
 		(pts
+			(xy 572.77 339.09) (xy 600.71 339.09)
+		)
+		(stroke
+			(width 0)
+			(type default)
+			(color 0 0 0 1)
+		)
+	)
+	(wire
+		(pts
 			(xy 67.31 386.08) (xy 69.85 386.08)
 		)
@@
 	(wire
 		(pts
+			(xy 542.29 321.31) (xy 541.02 321.31)
+		)
+		(stroke
+			(width 0)
+			(type default)
+		)
+	)
+	(wire
+		(pts
 			(xy 443.23 177.8) (xy 443.23 116.84)
 		)
@@
 	(wire
 		(pts
+			(xy 572.77 330.2) (xy 575.31 330.2)
+		)
+		(stroke
+			(width 0)
+			(type default)
+			(color 255 0 0 1)
+		)
+	)
+	(wire
+		(pts
 			(xy 509.27 88.9) (xy 521.97 88.9)
 		)
@@
 	(wire
 		(pts
+			(xy 541.02 297.18) (xy 546.1 297.18)
+		)
+		(stroke
+			(width 0)
+			(type default)
+		)
+	)
+	(wire
+		(pts
 			(xy 280.67 198.12) (xy 280.67 139.7)
 		)
@@
 				)
 			)
+		)
+	)
+	(sheet
+		(at 542.29 314.96)
+		(size 30.48 46.99)
+		(exclude_from_sim no)
+		(in_bom yes)
+		(on_board yes)
+		(dnp no)
+		(fields_autoplaced yes)
+		(stroke
+			(width 0.1524)
+			(type solid)
+		)
+		(fill
+			(color 0 0 0 0)
+		)
+		(property "Sheetname" "Variable Clock Module"
+			(at 542.29 314.2484 0)
+			(show_name no)
+			(do_not_autoplace no)
+			(effects
+				(font
+					(size 1.27 1.27)
+				)
+				(justify left bottom)
+			)
+		)
+		(property "Sheetfile" "clock.kicad_sch"
+			(at 542.29 362.5346 0)
+			(show_name no)
+			(do_not_autoplace no)
+			(effects
+				(font
+					(size 1.27 1.27)
+				)
+				(justify left top)
+			)
+		)
+		(pin "VCC" input
+			(at 572.77 330.2 0)
+			(effects
+				(font
+					(size 1.27 1.27)
+				)
+				(justify right)
+			)
+		)
+		(pin "CLK" output
+			(at 542.29 321.31 180)
+			(effects
+				(font
+					(size 1.27 1.27)
+				)
+				(justify left)
+			)
+		)
+		(pin "GND" input
+			(at 572.77 339.09 0)
+			(effects
+				(font
+					(size 1.27 1.27)
+				)
+				(justify right)
+			)
+		)
+		(instances
+			(project "Cykomputer"
+				(path "/7319cfd4-b54a-49cd-84bf-92265ba5acc0"
+					(page "3")
+				)
+			)
