File: Computer Designs/CYKEYBOARD/CYKEYBOARD.kicad_sch (KiCad schematic)
At the start: 355 parts, among them J1 Conn_01x12, J2 Conn_01x03, J3 Conn_01x03, K0 RESET, K1 F1, K10 F10, K11 F11, K12 F12, K13 READY, K14 ~~,,,,,,`, K15 !,,,,,,1, K16 @,,,,,,2, K17 #,,,,,,3, K18 $,,,,,,4, K19 #,,,,,,3, K2 F2, K20 ^,,,,,,6, K21 &,,,,,,7, K22 *,,,,,,8, K23 (,,,,,,9, K24 ),,,,,,0, K25 _,,,,,,-, K26 +,,,,,,=, K27 BACKSPACE, K28 INS, K29 HOME, K3 F3, K31 SAVE,,,,,,LOAD, K32 Q, K33 W, K34 E, K35 R, K36 T, K37 Y, K38 U, K39 I, K4 F4, K40 O, K41 P, K42 {,,,,,,[, K43 },,,,,,], K44 |,,,,,,\, K45 DEL, K46 HOLD, K48 SHIFT,,,,,,LOCK, K49 A, K5 F5, K50 S, K51 D, K52 F, K53 G, K54 H, K55 J, K56 K, K57 L, K58 :,,,,,,;, K59 ",,,,,,', K6 F6, K60 ENTER, K61 SHIFT, K62 Z, K63 X, K64 C, K65 V, K66 B, K67 N, K68 M, K69 <,,,,,,,, K7 F7, K70 >,,,,,,., K71 ?,,,,,,/, K72 SHIFT, K73 ^, K74 CTRL, K75 CYKA,,,,,,TECH, K76 ALT, K77 Blank, K78 ALT, K79 FN, K8 F8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

Commit message: Redesigning Keyboard
Parts:
- removed U1: 74HC154, PCM_Package_DIP_AKL:DIP-24_W7.62mm, symbol 74xx:74LS154
- removed U2: 74HC138, PCM_Package_DIP_AKL:DIP-16_W7.62mm, symbol 74xx:74HC138
- removed unit 1 of U3
- removed unit 2 of U3
- removed unit 4 of U5
- removed unit 1 of U5
- removed unit 2 of U5
- removed unit 3 of U5
- removed U6: 74HC374, Package_DIP:DIP-20_W7.62mm_Socket, symbol 74xx:74HC374
- removed Y1: ACO-xxxMHz-A, Oscillator:Oscillator_DIP-14, symbol Oscillator:ACO-xxxMHz-A
- added C15, C86, C87, C88, C89, C90, C91, C92, C93, C94, C95, C96: 1nF_Ceramic, Capacitor_THT:C_Disc_D5.0mm_W2.5mm_P2.50mm, symbol PCM_SL_Capacitors:1nF_Ceramic
- added D100, D97, D98, D99: D_Generic, symbol PCM_4ms_Diode:D_Generic
- added D30, D47, D86, D87, D88, D89, D90, D91, D92, D93, D94, D95: D, Diode_THT:D_T-1_P5.08mm_Horizontal, symbol Device:D
- added D96: LED, LED_THT:LED_D5.0mm, symbol PCM_SL_Devices:LED
- added K30: !,,,,,,1, Button_Switch_Keyboard:SW_Cherry_MX_1.00u_PCB, symbol Switch:SW_Push
- added K47: @,,,,,,2, Button_Switch_Keyboard:SW_Cherry_MX_1.00u_PCB, symbol Switch:SW_Push
- added K85: #,,,,,,3, Button_Switch_Keyboard:SW_Cherry_MX_1.00u_PCB, symbol Switch:SW_Push
- added K86: $,,,,,,4, Button_Switch_Keyboard:SW_Cherry_MX_1.00u_PCB, symbol Switch:SW_Push
- added K87: BACKSPACE, Button_Switch_Keyboard:SW_Cherry_MX_2.00u_PCB, symbol Switch:SW_Push
- added K88: ),,,,,,0, Button_Switch_Keyboard:SW_Cherry_MX_2.00u_PCB, symbol Switch:SW_Push
- added K89: %,,,,,,5, Button_Switch_Keyboard:SW_Cherry_MX_1.00u_PCB, symbol Switch:SW_Push
- added K90: ^,,,,,,6, Button_Switch_Keyboard:SW_Cherry_MX_1.00u_PCB, symbol Switch:SW_Push
- added K91: &,,,,,,7, Button_Switch_Keyboard:SW_Cherry_MX_1.00u_PCB, symbol Switch:SW_Push
- added K92: *,,,,,,8, Button_Switch_Keyboard:SW_Cherry_MX_1.00u_PCB, symbol Switch:SW_Push
- added K93: (,,,,,,9, Button_Switch_Keyboard:SW_Cherry_MX_1.00u_PCB, symbol Switch:SW_Push
- added K94: READY, Button_Switch_Keyboard:SW_Cherry_MX_2.75u_PCB, symbol Switch:SW_Push
- added R16, R87, R88, R89, R90, R91, R92, R93, R94, R95, R96, R97: 10k, Resistor_THT:R_Axial_DIN0207_L6.3mm_D2.5mm_P10.16mm_Horizontal, symbol PCM_SL_Resistors:10k
- added R17: 3.3k, Resistor_THT:R_Axial_DIN0207_L6.3mm_D2.5mm_P10.16mm_Horizontal, symbol PCM_SL_Resistors:3.3k
- added U2, U7: 74LS148, symbol 74xx:74LS148
- K19: value #,,,,,,3 -> %,,,,,,5
- R10, R11, R12, R13, R14, R15, R18, R19, R2, R20, R21, R22, R23, R24, R25, R26, R27, R28, R29, R3, R30, R31, R32, R33, R34, R35, R36, R37, R38, R39, R4, R40, R41, R42, R43, R44, R45, R46, R47, R48, R49, R5, R50, R51, R52, R53, R54, R55, R56, R57, R58, R59, R6, R60, R61, R62, R63, R64, R65, R66, R67, R68, R69, R7, R70, R71, R72, R73, R74, R75, R76, R77, R78, R79, R8, R80, R81, R82, R83, R85, R86, R9: value 4.7k -> 10k; symbol PCM_SL_Resistors:4.7k -> PCM_SL_Resistors:10k
Connections:
- net Col_0: now also U7.10 (IO)
- net Col_1: now also K30.1, U7.11 (I1)
- net Col_10: now also K88.1, U2.12 (I2)
- net Col_11: now also U2.13 (I3)
- net Col_12: now also U2.1 (I4)
- net Col_13: now also K87.1, U2.2 (I5)
- net Col_14: now also U2.3 (I6)
- net Col_15: now also U2.4 (I7)
- net Col_2: now also K47.1, U7.12 (I2)
- net Col_3: now also K85.1, U7.13 (I3)
- net Col_4: now also K86.1, U7.1 (I4)
- net Col_5: now also K89.1, U7.2 (I5)
- net Col_6: now also K90.1, U7.3 (I6)
- net Col_7: now also K91.1, U7.4 (I7)
- net Col_8: now also K92.1, U2.10 (IO)
- net Col_9: now also K93.1, U2.11 (I1)
- net GND: now also D96.1, K94.1, U2.8 (GND), U7.8 (GND); no longer U4.1, U4.5
- net Row_1: now also D30.1 (K), D47.1 (K), D86.1 (K), D87.1 (K), D88.1 (K), D89.1 (K), D90.1 (K), D91.1 (K), D92.1 (K), D93.1 (K), D94.1 (K)
- net VCC: now also R16.1, R17.1, R87.1, R88.1, R89.1, R90.1, R91.1, R92.1, R93.1, R94.1, R95.1, R96.1, R97.1, U2.16 (VCC), U7.16 (VCC)
- net IRQ: now reaches J1.2 (Pin_2)
- net IRQ: now also U4.6
- new net: C94.1, D92.2 (A), K91.2
- new net: C86.1, D30.2 (A), K30.2
- new net: C86.2, R87.2
- new net: C96.1, D94.2 (A), K93.2
- new net: C90.1, D88.2 (A), K87.2
- new net: C90.2, R91.2
- new net: C91.1, D89.2 (A), K88.2
- new net: C91.2, R92.2
- new net: C95.2, R96.2
- new net: C89.1, D87.2 (A), K86.2
- new net: C89.2, R90.2
- new net: C87.1, D47.2 (A), K47.2
- new net: C92.1, D90.2 (A), K89.2
- new net: C88.1, D86.2 (A), K85.2
- new net: C95.1, D93.2 (A), K92.2
- new net: C87.2, R88.2
- new net: D100.1 (K), D97.1 (K), D98.1 (K), D99.1 (K), U4.5
- new net: C15.1, D95.2 (A), K94.2
- new net: C15.2, R16.2
- new net: C96.2, R97.2
- new net: C93.1, D91.2 (A), K90.2
- new net: C92.2, R93.2
- new net: D96.2, R17.2
- new net: C93.2, R94.2
- new net: U2.5 (EI), U7.15 (EO)
- new net: C94.2, R95.2
- new net: C88.2, R89.2
- new net RDY_LOCK: D95.1 (K)
- no-connect marks 27 -> 12
Other:
- moved on the sheet: U4C

Commit message: changes
Parts:
- added U1, U10, U6, U9: 74HC04, symbol 74xx:74HC04
Connections:
- net Col_0: now also U9.9; no longer U7.10 (IO)
- net Col_1: now also U9.5; no longer U7.11 (I1)
- net Col_10: now also U1.13; no longer U2.12 (I2)
- net Col_11: now also U1.11; no longer U2.13 (I3)
- net Col_12: now also U1.9; no longer U2.1 (I4)
- net Col_13: now also U1.5; no longer U2.2 (I5)
- net Col_14: now also U1.3; no longer U2.3 (I6)
- net Col_15: now also U1.1; no longer U2.4 (I7)
- net Col_2: now also U9.3; no longer U7.12 (I2)
- net Col_3: now also U9.1; no longer U7.13 (I3)
- net Col_4: now also U6.13; no longer U7.1 (I4)
- net Col_5: now also U6.11; no longer U7.2 (I5)
- net Col_6: now also U6.9; no longer U7.3 (I6)
- net Col_7: now also U6.5; no longer U7.4 (I7)
- net Col_8: now also U6.3; no longer U2.10 (IO)
- net Col_9: now also U6.1; no longer U2.11 (I1)
- net GND: now also U1.7 (GND), U10.14 (VCC), U6.7 (GND), U9.7 (GND)
- net VCC: now also U1.14 (VCC), U10.7 (GND), U6.14 (VCC), U9.14 (VCC)
- net at U7.15 (EO): no longer U2.5 (EI)
- net at U7.5 (EI): now also U2.15 (EO)
- net at U7.6 (S2): now also U10.1
- net at U7.7 (S1): now also U10.3
- net at U7.9 (S0): now also U10.5
- net at U2.6 (S2): now also U9.11
- net at U2.7 (S1): now also U9.13
- net at U2.9 (S0): now also U10.9
- new net: U1.8, U2.1 (I4)
- new net: U2.10 (IO), U6.4
- new net: U6.10, U7.2 (I5)
- new net: U1.6, U2.2 (I5)
- new net: U6.12, U7.1 (I4)
- new net: U7.13 (I3), U9.2
- new net: U6.6, U7.4 (I7)
- new net: U7.11 (I1), U9.6
- new net: U1.10, U2.13 (I3)
- new net: U1.12, U2.12 (I2)
- new net: U6.8, U7.3 (I6)
- new net: U1.4, U2.3 (I6)
- new net: U7.10 (IO), U9.8
- new net: U7.12 (I2), U9.4
- new net: U2.11 (I1), U6.2
- new net: U1.2, U2.4 (I7)

Commit message: Continued
Parts:
- removed D100, D97, D98, D99: D_Generic, symbol PCM_4ms_Diode:D_Generic
- removed U1, U10, U6, U9: 74HC04, symbol 74xx:74HC04
- added U9: 74LS148, symbol 74xx:74LS148
Connections:
- net GND: now also J1.12 (Pin_12), R10.1, R11.1, R12.1, R13.1, R14.1, R15.1, R16.1, R18.1, R19.1, R2.1, R20.1, R21.1, R22.1, R23.1, R24.1, R25.1, R26.1, R27.1, R28.1, R29.1, R3.1, R30.1, R31.1, R32.1, R33.1, R34.1, R35.1, R36.1, R37.1, R38.1, R39.1, R4.1, R40.1, R41.1, R42.1, R43.1, R44.1, R45.1, R46.1, R47.1, R48.1, R49.1, R5.1, R50.1, R51.1, R52.1, R53.1, R54.1, R55.1, R56.1, R57.1, R58.1, R59.1, R6.1, R60.1, R61.1, R62.1, R63.1, R64.1, R65.1, R66.1, R67.1, R68.1, R69.1, R7.1, R70.1, R71.1, R72.1, R73.1, R74.1, R75.1, R76.1, R77.1, R78.1, R79.1, R8.1, R80.1, R81.1, R82.1, R83.1, R84.1, R85.1, R86.1, R87.1, R88.1, R89.1, R9.1, R90.1, R91.1, R92.1, R93.1, R94.1, R95.1, R96.1, R97.1; no longer J1.1 (Pin_1), K0.1, K13.1, K48.1
- net Row_0: now also U9.10 (IO)
- net Row_1: now also U9.11 (I1)
- net Row_2: now also U9.12 (I2)
- net Row_3: now also U9.13 (I3)
- net Row_4: now also U9.1 (I4)
- net Row_5: now also U9.2 (I5)
- net VCC: now also J1.1 (Pin_1), K0.1, K13.1, K48.1; no longer J1.12 (Pin_12), R10.1, R11.1, R12.1, R13.1, R14.1, R15.1, R16.1, R17.1, R18.1, R19.1, R2.1, R20.1, R21.1, R22.1, R23.1, R24.1, R25.1, R26.1, R27.1, R28.1, R29.1, R3.1, R30.1, R31.1, R32.1, R33.1, R34.1, R35.1, R36.1, R37.1, R38.1, R39.1, R4.1, R40.1, R41.1, R42.1, R43.1, R44.1, R45.1, R46.1, R47.1, R48.1, R49.1, R5.1, R50.1, R51.1, R52.1, R53.1, R54.1, R55.1, R56.1, R57.1, R58.1, R59.1, R6.1, R60.1, R61.1, R62.1, R63.1, R64.1, R65.1, R66.1, R67.1, R68.1, R69.1, R7.1, R70.1, R71.1, R72.1, R73.1, R74.1, R75.1, R76.1, R77.1, R78.1, R79.1, R8.1, R80.1, R81.1, R82.1, R83.1, R84.1, R85.1, R86.1, R87.1, R88.1, R89.1, R9.1, R90.1, R91.1, R92.1, R93.1, R94.1, R95.1, R96.1, R97.1, U8.4 (~{S})
- net at U4.4: now also U8.4 (~{S}); no longer U8.3 (C)
- net SHIFT_LED: now reaches U8.5 (Q)
- net SHIFT_LED: now also R17.1
Other:
- moved on the sheet: U4C

Commit message: Continued
Parts:
- added R100, R101, R102, R103, R104, R105, R106, R107, R108, R109, R110, R111, R112, R113, R98, R99: 10k, Resistor_THT:R_Axial_DIN0207_L6.3mm_D2.5mm_P10.16mm_Horizontal, symbol PCM_SL_Resistors:10k
Connections:
- net Col_0: now also U7.10 (IO), R113.1
- net Col_1: now also U7.11 (I1), R112.1
- net Col_10: now also U2.12 (I2), R103.1
- net Col_11: now also U2.13 (I3), R102.1
- net Col_12: now also U2.1 (I4), R101.1
- net Col_13: now also U2.2 (I5), R100.1
- net Col_14: now also U2.3 (I6), R99.1
- net Col_15: now also U2.4 (I7), R98.1
- net Col_2: now also U7.12 (I2), R111.1
- net Col_3: now also U7.13 (I3), R110.1
- net Col_4: now also U7.1 (I4), R109.1
- net Col_5: now also U7.2 (I5), R108.1
- net Col_6: now also U7.3 (I6), R107.1
- net Col_7: now also U7.4 (I7), R106.1
- net Col_8: now also U2.10 (IO), R105.1
- net Col_9: now also U2.11 (I1), R104.1
- net VCC: now also R100.2, R101.2, R102.2, R103.2, R104.2, R105.2, R106.2, R107.2, R108.2, R109.2, R110.2, R111.2, R112.2, R113.2, R98.2, R99.2

Commit message: Continued
Parts:
- added U1: 74HC14, symbol 74xx:74HC14
Connections:
- net GND: now also U1.7 (GND)
- net Row_0: now also U1.13; no longer U9.10 (IO)
- net Row_1: now also U1.11; no longer U9.11 (I1)
- net Row_2: now also U1.9; no longer U9.12 (I2)
- net Row_3: now also U1.5; no longer U9.13 (I3)
- net Row_4: now also U1.3; no longer U9.1 (I4)
- net Row_5: now also U1.1; no longer U9.2 (I5)
- net VCC: now also U1.14 (VCC)
- new net: U1.4, U9.1 (I4)
- new net: U1.12, U9.10 (IO)
- new net: U1.10, U9.11 (I1)
- new net: U1.8, U9.12 (I2)
- new net: U1.6, U9.13 (I3)
- new net: U1.2, U9.2 (I5)

Commit message: Continued
Parts:
- removed C10, C11, C12, C13, C2, C3, C4, C5, C6, C7, C8, C9: 1nF_Ceramic, Capacitor_THT:C_Disc_D5.0mm_W2.5mm_P2.50mm, symbol PCM_SL_Capacitors:1nF_Ceramic
- removed D1, D10, D11, D12, D2, D3, D4, D5, D6, D7, D8, D9: D, Diode_THT:D_T-1_P5.08mm_Horizontal, symbol Device:D
- removed K1: F1, Button_Switch_Keyboard:SW_Cherry_MX_1.00u_PCB, symbol Switch:SW_Push
- removed K10: F10, Button_Switch_Keyboard:SW_Cherry_MX_1.00u_PCB, symbol Switch:SW_Push
- removed K11: F11, Button_Switch_Keyboard:SW_Cherry_MX_1.00u_PCB, symbol Switch:SW_Push
- removed K12: F12, Button_Switch_Keyboard:SW_Cherry_MX_1.00u_PCB, symbol Switch:SW_Push
- removed K2: F2, Button_Switch_Keyboard:SW_Cherry_MX_1.00u_PCB, symbol Switch:SW_Push
- removed K3: F3, Button_Switch_Keyboard:SW_Cherry_MX_1.00u_PCB, symbol Switch:SW_Push
- removed K4: F4, Button_Switch_Keyboard:SW_Cherry_MX_1.00u_PCB, symbol Switch:SW_Push
- removed K5: F5, Button_Switch_Keyboard:SW_Cherry_MX_1.00u_PCB, symbol Switch:SW_Push
- removed K6: F6, Button_Switch_Keyboard:SW_Cherry_MX_1.00u_PCB, symbol Switch:SW_Push
- removed K7: F7, Button_Switch_Keyboard:SW_Cherry_MX_1.00u_PCB, symbol Switch:SW_Push
- removed K8: F8, Button_Switch_Keyboard:SW_Cherry_MX_1.00u_PCB, symbol Switch:SW_Push
- removed K9: F9, Button_Switch_Keyboard:SW_Cherry_MX_1.00u_PCB, symbol Switch:SW_Push
- removed R10, R11, R12, R13, R14, R3, R4, R5, R6, R7, R8, R9: 10k, Resistor_THT:R_Axial_DIN0207_L6.3mm_D2.5mm_P10.16mm_Horizontal, symbol PCM_SL_Resistors:10k
- removed U1: 74HC14, symbol 74xx:74HC14
- removed unit 3 of U4
- removed U8: 74HC74, Package_DIP:DIP-14_W7.62mm_Socket, symbol 74xx:74HC74
- added C100, C101, C102, C103, C104, C97, C98, C99: 1nF_Ceramic, Capacitor_THT:C_Disc_D5.0mm_W2.5mm_P2.50mm, symbol PCM_SL_Capacitors:1nF_Ceramic
- added D1, D2, D3, D4, D5, D6, D7, D8: D_Generic, symbol PCM_4ms_Diode:D_Generic
- added D100, D101, D102, D103, D104, D105, D106, D107, D108, D109, D110, D111, D112, D117, D118, D119, D120, D121, D122, D123, D124, D125, D126, D127, D128, D129, D130, D131, D132, D133, D134, D135, D136, D137, D138, D139, D140, D141, D142, D143, D144, D145, D146, D147, D148, D149, D150, D151, D152, D153, D154, D155, D156, D157, D158, D159, D160, D161, D162, D163, D164, D165, D166, D167, D168, D169, D170, D171, D172, D173, D174, D175, D176, D177, D178, D179, D180, D181, D182, D183, D97, D98, D99: D, Diode_THT:D_T-1_P5.08mm_Horizontal, symbol Device:D
- added D113: LED, LED_THT:LED_D5.0mm, symbol PCM_SL_Devices:LED
- added J4: Conn_01x09, 4ms_Connector:Pins_1x09_2.54mm_TH, symbol PCM_4ms_Connector:Conn_01x09
- added R115, R116, R117, R118, R119, R122, R123, R124, R125, R126, R127, R128, R129, R130, R131, R132, R133, R134, R135, R136, R137: 10k, Resistor_THT:R_Axial_DIN0207_L6.3mm_D2.5mm_P10.16mm_Horizontal, symbol PCM_SL_Resistors:10k
- added R120, R121, R138, R139, R140, R141: 2.2k, Resistor_THT:R_Axial_DIN0207_L6.3mm_D2.5mm_P10.16mm_Horizontal, symbol PCM_SL_Resistors:2.2k
- added R3, R4, R5, R6: 3.3k, Resistor_THT:R_Axial_DIN0207_L6.3mm_D2.5mm_P10.16mm_Horizontal, symbol PCM_SL_Resistors:3.3k
- added SW1, SW2, SW3, SW4, SW5, SW6, SW7, SW8: SW_Push, symbol Switch:SW_Push
- added U10, U11, U12, U13, U14, U15, U16, U6: 74HC14, Package_DIP:DIP-14_W7.62mm_Socket, symbol 74xx:74HC14
- added U17: 74HC14, symbol 74xx:74HC14
- added U8: 74LS76, Package_DIP:DIP-16_W7.62mm_Socket, symbol 74xx:74LS76
- added Y1: ACO-xxxMHz-A, Oscillator:Oscillator_DIP-14, symbol Oscillator:ACO-xxxMHz-A
- K87: footprint Button_Switch_Keyboard:SW_Cherry_MX_2.00u_PCB -> Button_Switch_Keyboard:SW_Cherry_MX_1.00u_PCB
- K94: footprint Button_Switch_Keyboard:SW_Cherry_MX_2.75u_PCB -> Button_Switch_Keyboard:SW_Cherry_MX_1.00u_PCB
- U2, U7, U9: footprint (none) -> Package_DIP:DIP-16_W7.62mm_Socket
Connections:
- net Row_4 is gone; now on net Col_0: D61.1 (K), D62.1 (K), D63.1 (K), D64.1 (K), D65.1 (K), D66.1 (K), D67.1 (K), D68.1 (K), D69.1 (K), D70.1 (K), D71.1 (K), D72.1 (K), D73.1 (K)
- net BIT0: now also D1.2 (A), U16.10
- net BIT1: now also D3.2 (A), U16.8
- net BIT2: now also D5.2 (A), U16.6
- net BIT3: now also D7.2 (A), U17.4
- net BIT4: now also D2.2 (A), U17.2
- net BIT5: now also D4.2 (A), U16.12
- net BIT6: now also D6.2 (A), U17.10
- net BIT7: now also D8.2 (A), U17.8
- net Col_0: now also D132.1 (K), D172.1 (K), D183.1 (K), D97.1 (K), D98.1 (K), R116.1, U15.11, U15.3, U8.14 (~{Q}); no longer K14.1, K31.1, K61.1, K72.1, K74.1, U7.10 (IO)
- net Col_1: now also D117.1 (K), D133.1 (K), D154.1 (K), D159.1 (K), D182.1 (K), U15.1; no longer K15.1, K30.1, K32.1, K49.1, K62.1, K75.1, U7.11 (I1)
- net Col_10: now also D126.1 (K), D142.1 (K), D157.1 (K), D168.1 (K), D173.1 (K), U13.9; no longer K24.1, K41.1, K58.1, K71.1, K88.1, U2.12 (I2)
- net Col_11: now also D127.1 (K), D143.1 (K), D169.1 (K), U13.5; no longer K25.1, K42.1, K59.1, U2.13 (I3)
- net Col_12: now also D104.1 (K), D128.1 (K), D144.1 (K), D170.1 (K), D171.1 (K), U13.3; no longer K26.1, K43.1, K60.1, K73.1, U2.1 (I4)
- net Col_13: now also D100.1 (K), D129.1 (K), D145.1 (K), D158.1 (K), D99.1 (K), U13.1; no longer K27.1, K44.1, K87.1, U2.2 (I5)
- net Col_14: now also D101.1 (K), D102.1 (K), D130.1 (K), D146.1 (K), U12.13; no longer K28.1, K45.1, U2.3 (I6)
- net Col_15: now also D103.1 (K), D131.1 (K), D147.1 (K), U12.11; no longer K29.1, K46.1, U2.4 (I7)
- net Col_2: now also D118.1 (K), D134.1 (K), D155.1 (K), D160.1 (K), D181.1 (K), U14.13; no longer K16.1, K33.1, K47.1, K50.1, K63.1, K76.1, K78.1, K81.1, U7.12 (I2)
- net Col_3: now also D119.1 (K), D135.1 (K), D156.1 (K), D161.1 (K), D180.1 (K), U14.11; no longer K17.1, K34.1, K51.1, K64.1, K77.1, K85.1, U7.13 (I3)
- net Col_4: now also D120.1 (K), D136.1 (K), D151.1 (K), D162.1 (K), D179.1 (K), U14.9; no longer K18.1, K35.1, K52.1, K65.1, K86.1, U7.1 (I4)
- net Col_5: now also D121.1 (K), D137.1 (K), D152.1 (K), D163.1 (K), D178.1 (K), U14.5; no longer K19.1, K36.1, K53.1, K66.1, K89.1, U7.2 (I5)
- net Col_6: now also D122.1 (K), D138.1 (K), D153.1 (K), D164.1 (K), D177.1 (K), U14.3; no longer K20.1, K37.1, K54.1, K67.1, K80.1, K90.1, U7.3 (I6)
- net Col_7: now also D123.1 (K), D139.1 (K), D148.1 (K), D165.1 (K), D176.1 (K), U14.1; no longer K21.1, K38.1, K55.1, K68.1, K91.1, U7.4 (I7)
- net Col_8: now also D124.1 (K), D140.1 (K), D149.1 (K), D166.1 (K), D175.1 (K), U13.13; no longer K22.1, K39.1, K56.1, K69.1, K92.1, U2.10 (IO)
- net Col_9: now also D125.1 (K), D141.1 (K), D150.1 (K), D167.1 (K), D174.1 (K), U13.11; no longer K23.1, K40.1, K57.1, K70.1, K93.1, U2.11 (I1)
- net GND: now also K0.1, K13.1, K14.1, K15.1, K16.1, K17.1, K18.1, K19.1, K20.1, K21.1, K22.1, K23.1, K24.1, K25.1, K26.1, K27.1, K28.1, K29.1, K30.1, K31.1, K32.1, K33.1, K34.1, K35.1, K36.1, K37.1, K38.1, K39.1, K40.1, K41.1, K42.1, K43.1, K44.1, K45.1, K46.1, K47.1, K48.1, K49.1, K50.1, K51.1, K52.1, K53.1, K54.1, K55.1, K56.1, K57.1, K58.1, K59.1, K60.1, K61.1, K62.1, K63.1, K64.1, K65.1, K66.1, K67.1, K68.1, K69.1, K70.1, K71.1, K72.1, K73.1, K74.1, K75.1, K76.1, K77.1, K78.1, K80.1, K81.1, K85.1, K86.1, K87.1, K88.1, K89.1, K90.1, K91.1, K92.1, K93.1, U9.8 (GND), D113.1, R3.1, SW1.1, SW2.1, SW3.1, SW4.1, SW5.1, SW6.1, SW7.1, SW8.1, U10.7 (GND), U11.11, U11.7 (GND), U12.7 (GND), U13.7 (GND), U14.7 (GND), U15.5, U15.7 (GND), U16.7 (GND), U17.13, U17.7 (GND), U6.7 (GND), U8.13 (GND), Y1.7 (GND); no longer R15.1, R18.1, R19.1, R2.1, R20.1, R21.1, R22.1, R23.1, R24.1, R25.1, R26.1, R29.1, R32.1, R33.1, R35.1, R36.1, R37.1, R38.1, R39.1, R40.1, R41.1, R42.1, R43.1, R44.1, R45.1, R46.1, R47.1, R48.1, R49.1, R50.1, R51.1, R52.1, R53.1, R54.1, R55.1, R56.1, R57.1, R58.1, R59.1, R60.1, R61.1, R62.1, R63.1, R64.1, R65.1, R66.1, R67.1, R68.1, R69.1, R70.1, R71.1, R72.1, R73.1, R74.1, R75.1, R76.1, R77.1, R78.1, R79.1, R80.1, R81.1, R82.1, R83.1, R84.1, R85.1, R86.1, R87.1, R88.1, R89.1, R90.1, R91.1, R92.1, R93.1, R94.1, R95.1, R96.1, R97.1, U4.13, U4.9
- net IRQ: now also D1.1 (K), D2.1 (K), D3.1 (K), D4.1 (K), D5.1 (K), D6.1 (K), D7.1 (K), D8.1 (K), R3.2
- net RDY_LOCK: now also U4.1
- net Row_0: now also D74.1 (K), D75.1 (K), D76.1 (K), D77.1 (K), D78.1 (K), D81.1 (K)
- net Row_1: now also R119.1, U16.3
- net Row_2: now also R118.1, U16.1
- net Row_3: now also D80.1 (K), R117.1, U15.13
- net Row_5: now also R115.1, U15.9; no longer D74.1 (K), D75.1 (K), D76.1 (K), D77.1 (K), D78.1 (K), D80.1 (K), D81.1 (K)
- net SHIFT_LED: now also U8.15 (Q)
- net SHIFT_LOCK: now also R5.1
- net VCC: now also R15.1, R18.1, R19.1, R2.1, R20.1, R21.1, R22.1, R23.1, R24.1, R25.1, R26.1, R29.1, R32.1, R33.1, R35.1, R36.1, R37.1, R38.1, R39.1, R40.1, R41.1, R42.1, R43.1, R44.1, R45.1, R46.1, R47.1, R48.1, R49.1, R50.1, R51.1, R52.1, R53.1, R54.1, R55.1, R56.1, R57.1, R58.1, R59.1, R60.1, R61.1, R62.1, R63.1, R64.1, R65.1, R66.1, R67.1, R68.1, R69.1, R70.1, R71.1, R72.1, R73.1, R74.1, R75.1, R76.1, R77.1, R78.1, R79.1, R80.1, R81.1, R82.1, R83.1, R84.1, R85.1, R86.1, R87.1, R88.1, R89.1, R90.1, R91.1, R92.1, R93.1, R94.1, R95.1, R96.1, R97.1, U9.16 (VCC), U9.2 (I5), U9.3 (I6), U9.4 (I7), R115.2, R116.2, R117.2, R118.2, R119.2, R120.2, R121.2, R122.1, R123.1, R124.1, R125.1, R126.2, R127.2, R128.2, R129.2, R130.2, R131.2, R132.2, R133.2, R134.1, R135.1, R136.1, R137.1, R138.2, R139.2, R140.2, R141.2, R4.2, R5.2, U10.14 (VCC), U11.14 (VCC), U12.14 (VCC), U13.14 (VCC), U14.14 (VCC), U15.14 (VCC), U16.14 (VCC), U17.14 (VCC), U6.14 (VCC), U8.5 (VCC), Y1.14 (Vcc); no longer K0.1, K13.1, K48.1
- net at C72.1, D77.2 (A), K77.2: now also D98.2 (A)
- net at C94.1, D92.2 (A), K91.2: now also D148.2 (A)
- net at C41.1, D70.2 (A), K70.2: now also D174.2 (A)
- net at C86.1, D30.2 (A), K30.2: now also D154.2 (A)
- net at C21.1, D27.2 (A), K27.2: now also D129.2 (A)
- net at C85.1, D14.2 (A), K14.2: now also D97.2 (A)
- net at C67.1, D34.2 (A), K34.2: now also D135.2 (A)
- net at C47.1, D68.2 (A), K68.2: now also D176.2 (A)
- net at C63.1, D52.2 (A), K52.2: now also D162.2 (A)
- net at C68.1, D51.2 (A), K51.2: now also D161.2 (A)
- net at C50.1, D22.2 (A), K22.2: now also D124.2 (A)
- net at C74.1, D50.2 (A), K50.2: now also D160.2 (A)
- net at C49.1, D23.2 (A), K23.2: now also D125.2 (A)
- net at C57.1, D37.2 (A), K37.2: now also D138.2 (A)
- net at C48.1, D39.2 (A), K39.2: now also D140.2 (A)
- net at C43.1, D69.2 (A), K69.2: now also D175.2 (A)
- net at C96.1, D94.2 (A), K93.2: now also D150.2 (A)
- net at C90.1, D88.2 (A), K87.2: now also D158.2 (A)
- net at C91.1, D89.2 (A), K88.2: now also D157.2 (A)
- net at C39.1, D41.2 (A), K41.2: now also D142.2 (A)
- net at C46.1, D56.2 (A), K56.2: now also D166.2 (A)
- net at C70.1, D63.2 (A), K63.2: now also D181.2 (A)
- net at C84.1, D31.2 (A), K31.2: now also D132.2 (A)
- net at C79.1, D49.2 (A), K49.2: now also D159.2 (A)
- net at C55.1, D54.2 (A), K54.2: now also D164.2 (A)
- net at C36.1, D42.2 (A), K42.2: now also D143.2 (A)
- net at C78.1, D32.2 (A), K32.2: now also D133.2 (A)
- net at C82.1, D61.2 (A), K61.2: now also D183.2 (A)
- net at C65.1, D18.2 (A), K18.2: now also D120.2 (A)
- net at C54.1, D67.2 (A), K67.2: now also D177.2 (A)
- net at C37.1, D25.2 (A), K25.2: now also D127.2 (A)
- net at C89.1, D87.2 (A), K86.2: now also D151.2 (A)
- net at C87.1, D47.2 (A), K47.2: now also D155.2 (A)
- net at C40.1, D58.2 (A), K58.2: now also D168.2 (A)
- net at C76.1, D16.2 (A), K16.2: now also D118.2 (A)
- net at C92.1, D90.2 (A), K89.2: now also D152.2 (A)
- net at C59.1, D19.2 (A), K19.2: now also D121.2 (A)
- net at C71.1, D76.2 (A), K76.2: now also D102.2 (A)
- net at C45.1, D40.2 (A), K40.2: now also D141.2 (A)
- net at C58.1, D20.2 (A), K20.2: now also D122.2 (A)
- net at C20.1, D45.2 (A), K45.2: now also D146.2 (A)
- net at C19.1, D28.2 (A), K28.2: now also D130.2 (A)
- net at C81.1, D74.2 (A), K74.2: now also D99.2 (A)
- net at C80.1, D75.2 (A), K75.2: now also D103.2 (A)
- net at C88.1, D86.2 (A), K85.2: now also D156.2 (A)
- net at C53.1, D55.2 (A), K55.2: now also D165.2 (A)
- net at C64.1, D35.2 (A), K35.2: now also D136.2 (A)
- net at U4.8: now also J3.2 (Pin_2)
- net at C52.1, D38.2 (A), K38.2: now also D139.2 (A)
- net at C95.1, D93.2 (A), K92.2: now also D149.2 (A)
- net at C51.1, D21.2 (A), K21.2: now also D123.2 (A)
- net at C44.1, D57.2 (A), K57.2: now also D167.2 (A)
- net at C73.1, D62.2 (A), K62.2: now also D182.2 (A)
- net at U4.2: now also U4.13
- net at C18.1, D29.2 (A), K29.2: now also D131.2 (A)
- net at C61.1, D53.2 (A), K53.2: now also D163.2 (A)
- net at C60.1, D36.2 (A), K36.2: now also D137.2 (A)
- net at U9.1 (I4): now also U11.12
- net at U9.10 (IO): now also U12.8
- net at U9.11 (I1): now also U12.6
- net at U9.12 (I2): now also U12.4
- net at U9.13 (I3): now also U12.2
- net at U9.6 (S2): now also U17.5
- net at U9.7 (S1): now also U17.9
- net at U9.9 (S0): now also U17.11
- net at C35.1, D59.2 (A), K59.2: now also D169.2 (A)
- net at C38.1, D24.2 (A), K24.2: now also D126.2 (A)
- net at C25.1, D26.2 (A), K26.2: now also D128.2 (A)
- net at C17.1, D46.2 (A), K46.2: now also D147.2 (A)
- net at C30.1, D81.2 (A), K81.2: now also D100.2 (A)
- net at C62.1, D65.2 (A), K65.2: now also D179.2 (A)
- net at C34.1, D71.2 (A), K71.2: now also D173.2 (A)
- net at C24.1, D43.2 (A), K43.2: now also D144.2 (A)
- net at C56.1, D66.2 (A), K66.2: now also D178.2 (A)
- net at C77.1, D15.2 (A), K15.2: now also D117.2 (A)
- net at C22.1, D44.2 (A), K44.2: now also D145.2 (A)
- net at C93.1, D91.2 (A), K90.2: now also D153.2 (A)
- net at C69.1, D64.2 (A), K64.2: now also D180.2 (A)
- net at C31.1, D72.2 (A), K72.2: now also D172.2 (A)
- net at U4.4: now also R120.1, U8.16 (K), U8.4 (J)
- net at C42.1, D78.2 (A), K78.2: now also D101.2 (A)
- net at C66.1, D17.2 (A), K17.2: now also D119.2 (A)
- net at C23.1, D60.2 (A), K60.2: now also D170.2 (A)
- net at C28.1, D73.2 (A), K73.2: now also D171.2 (A)
- net at U7.5 (EI): no longer U2.15 (EO)
- net at U7.6 (S2): now also U16.13
- net at U7.7 (S1): now also U17.1
- net at U7.9 (S0): now also U17.3
- net at C75.1, D33.2 (A), K33.2: now also D134.2 (A)
- net at U2.6 (S2): now also U16.5
- net at U2.7 (S1): now also U16.9
- net at U2.9 (S0): now also U16.11
- net at U4.12: now also R121.1, U8.12 (K), U8.9 (J)
- net RDY renamed PAUSE_LED
- net PAUSE_LED: now also U4.9, R4.1, R6.1, U8.11 (Q); no longer J3.2 (Pin_2)
- new net: U12.1, U15.10
- new net: R138.1, U8.3 (~{R})
- new net: C97.1, D105.2 (A), SW4.2
- new net: U11.13, U15.8
- new net: U8.1 (C), U8.6 (C), Y1.8 (OUT)
- new net: R139.1, U8.2 (~{S})
- new net: C99.2, R124.2
- new net: U12.10, U6.1
- new net: C103.1, D111.2 (A), SW7.2
- new net: C103.2, R136.2
- new net: U10.12, U7.1 (I4)
- new net: U10.13, U14.8
- new net: U10.8, U7.3 (I6)
- new net: U10.9, U14.4
- new net: C99.1, D107.2 (A), SW2.2
- new net: U11.1, U14.10
- new net: U11.2, U7.13 (I3)
- new net: D113.2, R6.2
- new net: U2.12 (I2), U6.12
- new net: U13.8, U6.13
- new net: C104.1, D112.2 (A), SW8.2
- new net: U10.3, U13.12
- new net: U10.4, U2.10 (IO)
- new net: C102.1, D110.2 (A), SW6.2
- new net: C102.2, R135.2
- new net: U11.9, U15.4
- new net: R141.1, U8.7 (~{S})
- new net: R140.1, U8.8 (~{R})
- new net: U11.3, U14.12
- new net: U10.5, U14.2
- new net: C98.2, R123.2
- new net: C98.1, D106.2 (A), SW3.2
- new net: U12.12, U6.3
- new net: U2.3 (I6), U6.4
- new net: U10.6, U7.4 (I7)
- new net: C100.1, D108.2 (A), SW1.2
- new net: U13.4, U6.9
- new net: U2.13 (I3), U6.10
- new net: U13.6, U6.11
- new net: U2.1 (I4), U6.8
- new net: U10.1, U13.10
- new net: U12.9, U16.4
- new net: U13.2, U6.5
- new net: U2.2 (I5), U6.6
- new net: U11.8, U7.10 (IO)
- new net: U12.3, U15.12
- new net: U10.10, U7.2 (I5)
- new net: U10.11, U14.6
- new net: U10.2, U2.11 (I1)
- new net: U12.5, U16.2
- new net: C104.2, R137.2
- new net: C101.1, D109.2 (A), SW5.2
- new net: C101.2, R134.2
- new net: U11.6, U7.11 (I1)
- new net: U11.4, U7.12 (I2)
- new net: C100.2, R125.2
- new net: C97.2, R122.2
- new net: U2.4 (I7), U6.2
- new net: U11.5, U15.2
- new net FB0: D105.1 (K), D106.1 (K), D107.1 (K), D108.1 (K), D109.1 (K), D110.1 (K), D111.1 (K), D112.1 (K), J4.1 (Pin_1), J4.2 (Pin_2), J4.3 (Pin_3), J4.4 (Pin_4), J4.5 (Pin_5), J4.6 (Pin_6), J4.7 (Pin_7), J4.8 (Pin_8), R126.1, R127.1, R128.1, R129.1, R130.1, R131.1, R132.1, R133.1
- no-connect marks 12 -> 10
Other:
- moved on the sheet: D85, R1, R100, R101, R102, R103, R104, R105, R106, R107, R108, R109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

Commit message: Continued
Parts:
- removed U3: 74HC393, PCM_Package_DIP_AKL:DIP-14_W7.62mm, symbol 74xx:74LS393
- removed U5: 74HC00, Package_DIP:DIP-14_W7.62mm_Socket, symbol 74xx:74HC00
- added D114, D115, D116, D184, D185, D186, D187, D188, D189, D190, D191, D192, D193, D194, D195, D196, D197, D198, D199, D200, D201, D202, D203, D204, D205, D206, D207, D208, D209, D210, D211, D212, D213, D214, D215, D216, D217, D218: D, Diode_THT:D_T-1_P5.08mm_Horizontal, symbol Device:D
- added U1: 74HC14, Package_DIP:DIP-14_W7.62mm_Socket, symbol 74xx:74HC14
- added unit 3 of U4
- D1, D2, D3, D4, D5, D6, D7, D8: footprint (none) -> Diode_THT:D_DO-35_SOD27_P7.62mm_Horizontal
- J4: footprint 4ms_Connector:Pins_1x09_2.54mm_TH -> Connector_Molex:Molex_SL_171971-0009_1x09_P2.54mm_Vertical
- SW1: value SW_Push -> F1; footprint (none) -> Button_Switch_Keyboard:SW_Cherry_MX_2.00u_PCB
- SW2: value SW_Push -> F2; footprint (none) -> Button_Switch_Keyboard:SW_Cherry_MX_2.00u_PCB
- SW3: value SW_Push -> F3; footprint (none) -> Button_Switch_Keyboard:SW_Cherry_MX_2.00u_PCB
- SW4: value SW_Push -> F4; footprint (none) -> Button_Switch_Keyboard:SW_Cherry_MX_2.00u_PCB
- SW5: value SW_Push -> F5; footprint (none) -> Button_Switch_Keyboard:SW_Cherry_MX_2.00u_PCB
- SW6: value SW_Push -> F6; footprint (none) -> Button_Switch_Keyboard:SW_Cherry_MX_2.00u_PCB
- SW7: value SW_Push -> F7; footprint (none) -> Button_Switch_Keyboard:SW_Cherry_MX_2.00u_PCB
- SW8: value SW_Push -> F8; footprint (none) -> Button_Switch_Keyboard:SW_Cherry_MX_2.00u_PCB
- U17: footprint (none) -> Package_DIP:DIP-14_W7.62mm_Socket
Connections:
- net Col_0: now also D202.1 (K); no longer D61.1 (K), D62.1 (K), D63.1 (K), D64.1 (K), D65.1 (K), D66.1 (K), D67.1 (K), D68.1 (K), D69.1 (K), D70.1 (K), D71.1 (K), D72.1 (K), D73.1 (K), R116.1, U15.11, U8.14 (~{Q})
- net Col_10: now also D116.1 (K); no longer K84.1
- net Col_5: now also D184.1 (K); no longer K79.1
- net Col_8: now also D114.1 (K); no longer K82.1
- net Col_9: now also D115.1 (K); no longer K83.1
- net FB0: now also D185.1 (K), D193.1 (K), D200.1 (K); no longer D105.1 (K), D106.1 (K), D107.1 (K), D108.1 (K), D109.1 (K), D110.1 (K), D111.1 (K), D112.1 (K), J4.2 (Pin_2), J4.3 (Pin_3), J4.4 (Pin_4), J4.5 (Pin_5), J4.6 (Pin_6), J4.7 (Pin_7), J4.8 (Pin_8), R127.1, R128.1, R129.1, R130.1, R131.1, R132.1, R133.1
- net GND: now also K79.1, K82.1, K83.1, K84.1, U1.11, U1.13, U1.5, U1.7 (GND), U1.9; no longer R16.1, R27.1, R28.1, R30.1, R31.1, R34.1, U11.11, U15.5, U17.13, U4.11
- net VCC: now also R16.1, R27.1, R28.1, R30.1, R31.1, R34.1, U1.14 (VCC)
- net at C32.1, D80.2 (A), K80.2: now also D104.2 (A)
- net at C26.1, D84.2 (A), K84.2: now also D116.2 (A)
- net at C27.1, D83.2 (A), K83.2: now also D115.2 (A)
- net at C33.1, D79.2 (A), K79.2: now also D184.2 (A)
- net at C29.1, D82.2 (A), K82.2: now also D114.2 (A)
- net at U9.6 (S2): no longer U17.5
- net at U15.6: now also D199.2 (A), D214.2 (A), D215.2 (A), D216.2 (A), D217.2 (A), D218.2 (A)
- net at U11.10: now also D200.2 (A), D208.2 (A), D209.2 (A), D210.2 (A), D211.2 (A), D212.2 (A), D213.2 (A)
- net at U17.12: now also D198.2 (A)
- net at U17.6: now also D195.2 (A)
- net at U4.10: now also D194.2 (A)
- new net: D186.2 (A), D187.2 (A), D188.2 (A), D189.2 (A), D190.2 (A), D191.2 (A), D192.2 (A), D193.2 (A), D194.1 (K), D195.1 (K), D196.1 (K), D197.1 (K), D198.1 (K)
- new net: D201.2 (A), D202.2 (A), U8.14 (~{Q})
- new net: D107.1 (K), U15.5
- new net: D185.2 (A), D203.2 (A), D204.2 (A), D205.2 (A), D206.2 (A), D207.2 (A), U4.6
- new net: D196.2 (A), U1.2
- new net: D110.1 (K), U1.1
- new net: D108.1 (K), U17.13
- new net: D106.1 (K), U11.11
- new net: D105.1 (K), U4.5
- new net: D197.2 (A), U1.4
- new net: D109.1 (K), U1.3
- new net: D112.1 (K), U4.11
- new net: D111.1 (K), U17.5
- new net FB1: D192.1 (K), D203.1 (K), D208.1 (K), J4.2 (Pin_2), R127.1
- new net FB2: D191.1 (K), J4.3 (Pin_3), R128.1
- new net FB3: D190.1 (K), D209.1 (K), J4.4 (Pin_4), R129.1
- new net FB4: D189.1 (K), D204.1 (K), D210.1 (K), J4.5 (Pin_5), R130.1
- new net FB5: D188.1 (K), D205.1 (K), D211.1 (K), J4.6 (Pin_6), R131.1
- new net FB6: D187.1 (K), D206.1 (K), D212.1 (K), J4.7 (Pin_7), R132.1
- new net FB7: D186.1 (K), D207.1 (K), D213.1 (K), J4.8 (Pin_8), R133.1
- new net Row_4: D201.1 (K), D61.1 (K), D62.1 (K), D63.1 (K), D64.1 (K), D65.1 (K), D66.1 (K), D67.1 (K), D68.1 (K), D69.1 (K), D70.1 (K), D71.1 (K), D72.1 (K), D73.1 (K), R116.1, U15.11
- no-connect marks 10 -> 20
Other:
- moved on the sheet: U11E, U14G, U15C, U15G, U17C, U17F, U4E

Commit message: Continued
Parts:
- removed D186, D187, D188, D189, D190, D191, D192, D193: D, Diode_THT:D_T-1_P5.08mm_Horizontal, symbol Device:D
- added D219, D220, D221, D222, D223, D224, D225, D226, D227, D228, D229, D230, D231, D232, D233, D234, D235, D236, D237, D238, D239, D240, D241: D, Diode_THT:D_T-1_P5.08mm_Horizontal, symbol Device:D
- D1, D2, D3, D4, D5, D6, D7, D8: value D_Generic -> D; symbol PCM_4ms_Diode:D_Generic -> Device:D
Connections:
- net Row_0 is gone; now on net Row_5: D74.1 (K), D75.1 (K), D76.1 (K), D77.1 (K), D78.1 (K), D81.1 (K)
- net FB0: now also D194.1 (K), D199.1 (K), J4.9 (Pin_9); no longer J4.1 (Pin_1)
- net FB1: now also D198.1 (K), J4.8 (Pin_8); no longer J4.2 (Pin_2)
- net FB2: now also D195.1 (K), D196.1 (K), D197.1 (K), J4.7 (Pin_7), D224.1 (K); no longer J4.3 (Pin_3)
- net FB3: now also D214.1 (K), J4.6 (Pin_6), D219.1 (K), D229.1 (K), D237.1 (K); no longer J4.4 (Pin_4)
- net FB4: now also D215.1 (K), D220.1 (K), D225.1 (K), D230.1 (K), D233.1 (K), D238.1 (K)
- net FB5: now also D216.1 (K), J4.4 (Pin_4), D221.1 (K), D226.1 (K), D231.1 (K), D234.1 (K), D239.1 (K); no longer J4.6 (Pin_6)
- net FB6: now also D217.1 (K), J4.3 (Pin_3), D222.1 (K), D227.1 (K), D232.1 (K), D235.1 (K), D240.1 (K); no longer J4.7 (Pin_7)
- net FB7: now also D218.1 (K), J4.2 (Pin_2), D223.1 (K), D228.1 (K), D236.1 (K), D241.1 (K); no longer J4.8 (Pin_8)
- net at D196.2 (A), U1.2: now also D233.2 (A), D234.2 (A), D235.2 (A), D236.2 (A)
- net at D198.2 (A), U17.12: now also D219.2 (A), D220.2 (A), D221.2 (A), D222.2 (A), D223.2 (A)
- net at D194.2 (A), U4.10: now also D224.2 (A), D225.2 (A), D226.2 (A), D227.2 (A), D228.2 (A)
- net at D197.2 (A), U1.4: now also D237.2 (A), D238.2 (A), D239.2 (A), D240.2 (A), D241.2 (A)
- net at D195.2 (A), U17.6: now also D229.2 (A), D230.2 (A), D231.2 (A), D232.2 (A)
Other:
- moved on the sheet: J4
