File: Computer Designs/CYKEYBOARD/CYKEYBOARD.kicad_sch (KiCad schematic)
At the start: 574 parts, among them J1 Conn_01x12, J2 Conn_01x03, J3 Conn_01x03, J4 Conn_01x09, K0 RESET, K13 READY, K14 ~~,,,,,,`, K15 !,,,,,,1, K16 @,,,,,,2, K17 #,,,,,,3, K18 $,,,,,,4, K19 %,,,,,,5, K20 ^,,,,,,6, K21 &,,,,,,7, K22 *,,,,,,8, K23 (,,,,,,9, K24 ),,,,,,0, K25 _,,,,,,-, K26 +,,,,,,=, K27 BACKSPACE, K28 INS, K29 HOME, K30 !,,,,,,1, K31 SAVE,,,,,,LOAD, K32 Q, K33 W, K34 E, K35 R, K36 T, K37 Y, K38 U, K39 I, K40 O, K41 P, K42 {,,,,,,[, K43 },,,,,,], K44 |,,,,,,\, K45 DEL, K46 HOLD, K47 @,,,,,,2, K48 SHIFT,,,,,,LOCK, K49 A, K50 S, K51 D, K52 F, K53 G, K54 H, K55 J, K56 K, K57 L, K58 :,,,,,,;, K59 ",,,,,,', K60 ENTER, K61 SHIFT, K62 Z, K63 X, K64 C, K65 V, K66 B, K67 N, K68 M, K69 <,,,,,,,, K70 >,,,,,,., K71 ?,,,,,,/, K72 SHIFT, K73 ^, K74 CTRL, K75 CYKA,,,,,,TECH, K76 ALT, K77 Blank, K78 ALT, K79 FN, K80 SELECT, K81 CTRL, K82 <, K83 \/, K84 >, K85 #,,,,,,3, K86 $,,,,,,4, K87 BACKSPACE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

Commit message: Continued
Parts:
- K28: value INS -> HOME
- K29: value HOME -> MON
- K46: value HOLD -> BAS
- K94: value READY -> PAUSE
Changed lines of the file:
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@@
 			)
 		)
-		(property "Value" "INS"
+		(property "Value" "HOME"
 			(at 340.36 41.91 0)
 			(hide yes)
@@
 			)
 		)
-		(property "Value" "HOME"
+		(property "Value" "MON"
 			(at 360.68 41.91 0)
 			(hide yes)
@@
 			)
 		)
-		(property "Value" "READY"
+		(property "Value" "PAUSE"
 			(at 378.46 41.91 0)
 			(hide yes)
@@
 			)
 		)
-		(property "Value" "HOLD"
+		(property "Value" "BAS"
 			(at 360.68 54.61 0)
 			(hide yes)

Commit message: Continued
Parts:
- added D186, D187: D, Diode_THT:D_T-1_P5.08mm_Horizontal, symbol Device:D
- added R114, R142, R143, R144: 10k, Resistor_THT:R_Axial_DIN0207_L6.3mm_D2.5mm_P10.16mm_Horizontal, symbol PCM_SL_Resistors:10k
- added U3: 7408, symbol 74xx_IEEE:7408
Connections:
- net Col_15: now also R114.2, R143.2, U3.1, U3.4
- net GND: now also U3.10, U3.12, U3.13, U3.7 (GND), U3.7 (GND), U3.9
- net Row_1: now also R144.2, U3.2
- net Row_2: now also R142.2, U3.5
- net VCC: now also R114.1, R142.1, R143.1, R144.1, U3.14 (VCC), U3.14 (VCC)
- net NMI: now reaches J1.11 (Pin_11)
- net NMI: now also D186.1 (K), D187.1 (K)
- new net: D186.2 (A), U3.6
- new net: D187.2 (A), U3.3
- no-connect marks 20 -> 21

Commit message: Finished Keyboard Design
Parts:
- removed R139, R141: 2.2k, Resistor_THT:R_Axial_DIN0207_L6.3mm_D2.5mm_P10.16mm_Horizontal, symbol PCM_SL_Resistors:2.2k
- U1, U10, U11, U12, U13, U14, U15, U16, U17, U4, U6: value 74HC14 -> 74LS14
- U3: value 7408 -> 74LS08; footprint (none) -> Package_DIP:DIP-14_W7.62mm_Socket
- U8: value 74LS76 -> 74LS107; footprint Package_DIP:DIP-16_W7.62mm_Socket -> Package_DIP:DIP-14_W7.62mm_Socket; symbol 74xx:74LS76 -> 74xx:74LS107
- Y1: value ACO-xxxMHz-A -> ACO-1MHz-A
Connections:
- net GND: now also U8.7 (GND); no longer U8.13 (GND)
- net PAUSE_LED: now also U8.5 (Q); no longer U8.11 (Q)
- net SHIFT_LED: now also U8.3 (Q); no longer U8.15 (Q)
- net VCC: now also U8.14 (VCC); no longer U8.5 (VCC)
- net at D201.2 (A), D202.2 (A): now also U8.2 (~{Q}); no longer U8.14 (~{Q})
- net at R138.1: now also U8.13 (~{R}); no longer U8.3 (~{R})
- net at R120.1, U4.4, U8.4 (K): now also U8.1 (J); no longer U8.16 (K)
- net at R121.1, U4.12: now also U8.11 (K), U8.8 (J); no longer U8.12 (K), U8.9 (J)
- net at U8.10 (~{R}): now also R140.1
- new net: U8.12 (C), U8.9 (C), Y1.8 (OUT)
- now unconnected: U8.6 (C)

Commit message: Added zeropage.s and msbasic.s, finished keyboard (really)
Connections:
- net GND: now also U2.5 (EI), U7.5 (EI), U9.5 (EI)
- no-connect marks 21 -> 18
Changed lines of the file:
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@@
 	)
 	(no_connect
-		(at 398.78 194.31)
-	)
-	(no_connect
 		(at 373.38 124.46)
 	)
@@
 	)
 	(no_connect
-		(at 398.78 119.38)
-	)
-	(no_connect
 		(at 35.56 140.97)
 	)
@@
 		(at 373.38 209.55)
 	)
-	(no_connect
-		(at 398.78 156.21)
-	)
 	(wire
 		(pts
@@
 		)
 	)
+	(label "GND"
+		(at 398.78 156.21 0)
+		(effects
+			(font
+				(size 1.27 1.27)
+			)
+			(justify left bottom)
+		)
+	)
 	(label "Row_1"
 		(at 424.18 86.36 0)
@@
 		)
 	)
+	(label "GND"
+		(at 398.78 194.31 0)
+		(effects
+			(font
+				(size 1.27 1.27)
+			)
+			(justify left bottom)
+		)
+	)
 	(label "Col_2"
 		(at 78.74 59.69 180)
@@
 		)
 	)
+	(label "GND"
+		(at 398.78 119.38 0)
+		(effects
+			(font
+				(size 1.27 1.27)
+			)
+			(justify left bottom)
+		)
+	)

Commit message: Continued
Parts:
- removed D185, D194, D195, D196, D197, D198, D199, D200, D203, D204, D205, D206, D207, D208, D209, D210, D211, D212, D213, D214, D215, D216, D217, D218, D219, D220, D221, D222, D223, D224, D225, D226, D227, D228, D229, D230, D231, D232, D233, D234, D235, D236, D237, D238, D239, D240, D241: D, Diode_THT:D_T-1_P5.08mm_Horizontal, symbol Device:D
- removed D4, D5, D6, D7, D8: D, Diode_THT:D_DO-35_SOD27_P7.62mm_Horizontal, symbol Device:D
- removed J4: Conn_01x09, Connector_Molex:Molex_SL_171971-0009_1x09_P2.54mm_Vertical, symbol PCM_4ms_Connector:Conn_01x09
- removed R126, R127, R128, R129, R130, R131, R132, R133: 10k, Resistor_THT:R_Axial_DIN0207_L6.3mm_D2.5mm_P10.16mm_Horizontal, symbol PCM_SL_Resistors:10k
- removed U1, U10, U11, U12, U13, U14, U15, U16, U17, U4, U6: 74LS14, Package_DIP:DIP-14_W7.62mm_Socket, symbol 74xx:74HC14
Connections:
- net BIT0: no longer D1.2 (A)
- net BIT1: no longer D3.2 (A)
- net BIT4: no longer D2.2 (A)
- net Col_1: now also D108.1 (K)
- net Col_12: now also D110.1 (K)
- net Col_2: now also D107.1 (K)
- net Col_3: now also D106.1 (K)
- net Col_4: now also D105.1 (K)
- net Col_6: now also D109.1 (K)
- net Col_7: now also D111.1 (K)
- net GS2: now reaches U9.14 (GS)
- net GS2: now also D2.2 (A)
- net GS1: now reaches U7.14 (GS)
- net GS1: now also D1.2 (A)
- net GS3: now reaches U2.14 (GS)
- net GS3: now also D3.2 (A)
- no-connect marks 18 -> 14

Commit message: Continued
Parts:
- added D185, D188, D189, D190, D191, D192, D193, D194: D, Diode_THT:D_T-1_P5.08mm_Horizontal, symbol Device:D
Connections:
- net Col_11: now also D112.1 (K)
- net GND: now also SW4.2; no longer SW4.1
- net Row_5: now also D185.1 (K), D188.1 (K), D189.1 (K), D190.1 (K), D191.1 (K), D192.1 (K), D193.1 (K), D194.1 (K)
- net at C97.1, D105.2 (A): now also SW4.1, D194.2 (A); no longer SW4.2
- net at C103.1, D111.2 (A), SW7.2: now also D188.2 (A)
- net at C99.1, D107.2 (A), SW2.2: now also D192.2 (A)
- net at C104.1, D112.2 (A), SW8.2: now also D185.2 (A)
- net at C102.1, D110.2 (A), SW6.2: now also D189.2 (A)
- net at C100.1, D108.2 (A), SW1.2: now also D191.2 (A)
- net at C101.1, D109.2 (A), SW5.2: now also D190.2 (A)

Commit message: Continued
Parts:
- removed unit 4 of U3
- removed unit 3 of U3
- added Q1, Q2: 2N2222A-TO92, PCM_Package_TO_SOT_THT_AKL:TO-92_Inline_Wide_EBC, symbol PCM_Transistor_BJT_AKL:2N2222A-TO92
Connections:
- net GND: now also R100.2, R101.2, R102.2, R103.2, R104.2, R105.2, R106.2, R107.2, R108.2, R109.2, R110.2, R111.2, R112.2, R113.2, R115.2, R116.2, R117.2, R118.2, R119.2, R98.2, R99.2; no longer U2.5 (EI), U7.5 (EI), U9.5 (EI)
- net GS1: now also U3.13; no longer D1.2 (A)
- net GS2: now also U3.10; no longer D2.2 (A)
- net GS3: now also Q2.2 (B); no longer D3.2 (A)
- net VCC: now also U3.14 (VCC), Q1.3 (C); no longer R100.2, R101.2, R102.2, R103.2, R104.2, R105.2, R106.2, R107.2, R108.2, R109.2, R110.2, R111.2, R112.2, R113.2, R115.2, R116.2, R117.2, R118.2, R119.2, R98.2, R99.2
- net EO2: now reaches U9.15 (EO)
- net EO2: now also Q1.2 (B)
- net EO1: now reaches U7.15 (EO)
- net EO1: now also U3.9
- net EO0: now reaches U2.15 (EO)
- net EO0: now also U3.12
- new net: D1.2 (A), U3.11
- new net: D2.2 (A), U3.8
- new net: D3.2 (A), Q2.1 (E)
- new net: Q1.1 (E), Q2.3 (C)
- no-connect marks 14 -> 9
Other:
- moved on the sheet: D1, D2, D3, R3

Commit message: Continued
Parts:
- added R7: 3.3k, Resistor_THT:R_Axial_DIN0207_L6.3mm_D2.5mm_P10.16mm_Horizontal, symbol PCM_SL_Resistors:3.3k
- added U1, U4: 74LS08, Package_DIP:DIP-14_W7.62mm_Socket, symbol 74xx:74LS08
- added U10, U13, U14: 74LS30, Package_DIP:DIP-14_W7.62mm_Socket, symbol 74xx:74LS30
- added U11, U5, U6: 74AHC541, Package_DIP:DIP-20_W7.62mm_Socket, symbol 74xx:74AHC541
- added U12: 74HC00, Package_DIP:DIP-14_W7.62mm_Socket, symbol 74xx:74HC00
- added U15: 74HC14, Package_DIP:DIP-14_W7.62mm_Socket, symbol 74xx:74HC14
- added unit 3 of U3
- added unit 4 of U3
Connections:
- net BIT0: now also U9.9 (S0)
- net BIT1: now also U9.7 (S1)
- net BIT2: now also U7.9 (S0)
- net BIT3: now also U7.7 (S1)
- net BIT4: now also U7.6 (S2)
- net BIT5: now also U2.9 (S0)
- net BIT6: now also U2.7 (S1)
- net BIT7: now also U2.6 (S2)
- net Col_0: now also U6.11 (Y7); no longer R113.1
- net Col_1: now also U6.12 (Y6); no longer R112.1
- net Col_10: now also U5.13 (Y5); no longer R103.1
- net Col_11: now also U5.14 (Y4); no longer R102.1
- net Col_12: now also U5.15 (Y3); no longer R101.1
- net Col_13: now also U5.16 (Y2); no longer R100.1
- net Col_14: now also U5.17 (Y1); no longer R99.1
- net Col_15: now also U5.18 (Y0); no longer R98.1
- net Col_2: now also U6.13 (Y5); no longer R111.1
- net Col_3: now also U6.14 (Y4); no longer R110.1
- net Col_4: now also U6.15 (Y3); no longer R109.1
- net Col_5: now also U6.16 (Y2); no longer R108.1
- net Col_6: now also U6.17 (Y1); no longer R107.1
- net Col_7: now also U6.18 (Y0); no longer R106.1
- net Col_8: now also U5.11 (Y7); no longer R105.1
- net Col_9: now also U5.12 (Y6); no longer R104.1
- net EO0: now also U12.1; no longer U3.12
- net EO1: now also U12.4; no longer U3.9
- net GND: now also Q1.3 (C), U3.7 (GND), U3.7 (GND), U1.7 (GND), U10.11, U10.12, U10.6, U10.7 (GND), U11.1 (G1), U11.10 (GND), U11.16 (Y2), U11.17 (Y1), U11.18 (Y0), U11.19 (G2), U12.10, U12.12, U12.13, U12.7 (GND), U12.9, U13.7 (GND), U14.7 (GND), U15.11, U15.13, U15.7 (GND), U3.10, U3.12, U3.13, U3.7 (GND), U3.7 (GND), U3.9, U4.7 (GND), U5.1 (G1), U5.19 (G2), U6.1 (G1), U6.10 (GND), U6.19 (G2), U6.20 (VCC); no longer R100.2, R101.2, R102.2, R103.2, R104.2, R105.2, R106.2, R107.2, R108.2, R109.2, R110.2, R111.2, R112.2, R113.2, R115.2, R116.2, R117.2, R118.2, R119.2, R3.1, R98.2, R99.2
- net GS1: now also U12.2; no longer U3.13
- net GS2: now also U12.5; no longer U3.10
- net PAUSE_LED: now also U15.5
- net RDY_LOCK: now also U15.3
- net Row_1: now also U11.11 (Y7); no longer R119.1
- net Row_2: now also U11.12 (Y6); no longer R118.1
- net Row_3: now also U11.13 (Y5); no longer R117.1
- net Row_4: now also U11.14 (Y4); no longer R116.1
- net Row_5: now also U11.15 (Y3); no longer R115.1
- net SHIFT_LOCK: now also U15.1
- net VCC: now also R100.2, R101.2, R102.2, R103.2, R104.2, R105.2, R106.2, R107.2, R108.2, R109.2, R110.2, R111.2, R112.2, R113.2, R115.2, R116.2, R117.2, R118.2, R119.2, R3.1, R98.2, R99.2, U3.14 (VCC), R7.2, U1.14 (VCC), U10.14 (VCC), U11.20 (VCC), U12.14 (VCC), U13.14 (VCC), U14.14 (VCC), U15.14 (VCC), U3.14 (VCC), U3.14 (VCC), U4.14 (VCC), U5.10 (GND), U5.20 (VCC); no longer Q1.3 (C)
- net at R120.1, U8.1 (J), U8.4 (K): now also U15.2
- net at D1.2 (A): now also U12.3; no longer U3.11
- net at D2.2 (A): now also U12.6; no longer U3.8
- net at D3.2 (A), Q2.1 (E): now also R7.1
- net at D193.2 (A): now also C98.1, D106.2 (A), SW3.2
- net at R121.1, U8.11 (K), U8.8 (J): now also U15.8
- net at U9.1 (I4): now also R115.1, U10.5, U11.5 (A3)
- net at U9.10 (IO): now also R119.1, U10.1, U11.9 (A7)
- net at U9.11 (I1): now also R118.1, U10.2, U11.8 (A6)
- net at U9.12 (I2): now also R117.1, U10.3, U11.7 (A5)
- net at U9.13 (I3): now also R116.1, U10.4, U11.6 (A4)
- net at U9.5 (EI): now also U10.8
- net at J3.2 (Pin_2): now also U15.6
- net BUF-C4: now reaches U7.1 (I4)
- net BUF-C4: now also R109.1, U1.12, U13.4, U6.5 (A3)
- net BUF-C0: now reaches U7.10 (IO)
- net BUF-C0: now also R113.1, U13.12, U4.12, U6.9 (A7)
- net BUF-C1: now reaches U7.11 (I1)
- net BUF-C1: now also R112.1, U13.11, U4.9, U6.8 (A6)
- net BUF-C2: now reaches U7.12 (I2)
- net BUF-C2: now also R111.1, U13.6, U4.4, U6.7 (A5)
- net BUF-C3: now reaches U7.13 (I3)
- net BUF-C3: now also R110.1, U13.5, U4.1, U6.6 (A4)
- net BUF-C5: now reaches U7.2 (I5)
- net BUF-C5: now also R108.1, U1.9, U13.3, U6.4 (A2)
- net BUF-C6: now reaches U7.3 (I6)
- net BUF-C6: now also R107.1, U1.4, U13.2, U6.3 (A1)
- net BUF-C7: now reaches U7.4 (I7)
- net BUF-C7: now also R106.1, U1.1, U13.1, U6.2 (A0)
- net at U7.5 (EI): now also U13.8
- net ADJ_C12: now reaches U2.1 (I4)
- net ADJ_C12: now also R101.1, U1.11, U1.13, U14.4, U5.5 (A3)
- net ADJ_C8: now reaches U2.10 (IO)
- net ADJ_C8: now also R105.1, U14.12, U4.11, U4.13, U5.9 (A7)
- net ADJ_C9: now reaches U2.11 (I1)
- net ADJ_C9: now also R104.1, U14.11, U4.10, U4.8, U5.8 (A6)
- net ADJ_C10: now reaches U2.12 (I2)
- net ADJ_C10: now also R103.1, U14.6, U4.5, U4.6, U5.7 (A5)
- net ADJ_C11: now reaches U2.13 (I3)
- net ADJ_C11: now also R102.1, U14.5, U4.2, U4.3, U5.6 (A4)
- net ADJ_C13: now reaches U2.2 (I5)
- net ADJ_C13: now also R100.1, U1.10, U1.8, U14.3, U5.4 (A2)
- net ADJ_C14: now reaches U2.3 (I6)
- net ADJ_C14: now also R99.1, U1.5, U1.6, U14.2, U5.3 (A1)
- net ADJ_C15: now reaches U2.4 (I7)
- net ADJ_C15: now also R98.1, U1.2, U1.3, U14.1, U5.2 (A0)
- net at U2.5 (EI): now also U14.8
- new net: U15.4, U15.9
- no-connect marks 9 -> 14
Other:
- moved on the sheet: U8C
