File: Computer Designs/CYKEYBOARD/CYKEYBOARD.kicad_sch (KiCad schematic)
At the start: 528 parts, among them J1 Conn_01x12, J2 Conn_01x03, J3 Conn_01x03, K0 RESET, K13 READY, K14 ~~,,,,,,`, K15 !,,,,,,1, K16 @,,,,,,2, K17 #,,,,,,3, K18 $,,,,,,4, K19 %,,,,,,5, K20 ^,,,,,,6, K21 &,,,,,,7, K22 *,,,,,,8, K23 (,,,,,,9, K24 ),,,,,,0, K25 _,,,,,,-, K26 +,,,,,,=, K27 BACKSPACE, K28 HOME, K29 MON, K30 !,,,,,,1, K31 SAVE,,,,,,LOAD, K32 Q, K33 W, K34 E, K35 R, K36 T, K37 Y, K38 U, K39 I, K40 O, K41 P, K42 {,,,,,,[, K43 },,,,,,], K44 |,,,,,,\, K45 DEL, K46 BAS, K47 @,,,,,,2, K48 SHIFT,,,,,,LOCK, K49 A, K50 S, K51 D, K52 F, K53 G, K54 H, K55 J, K56 K, K57 L, K58 :,,,,,,;, K59 ",,,,,,', K60 ENTER, K61 SHIFT, K62 Z, K63 X, K64 C, K65 V, K66 B, K67 N, K68 M, K69 <,,,,,,,, K70 >,,,,,,., K71 ?,,,,,,/, K72 SHIFT, K73 ^, K74 CTRL, K75 CYKA,,,,,,TECH, K76 ALT, K77 Blank, K78 ALT, K79 FN, K80 SELECT, K81 CTRL, K82 <, K83 \/, K84 >, K85 #,,,,,,3, K86 $,,,,,,4, K87 BACKSPACE, K88 ),,,,,,0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

Commit message: Continued
Parts:
- removed C1, C100, C101, C102, C103, C104, C14, C15, C17, C18, C19, C20, C21, C22, C23, C24, C25, C26, C27, C28, C29, C30, C31, C32, C33, C34, C35, C36, C37, C38, C39, C40, C41, C42, C43, C44, C45, C46, C47, C48, C49, C50, C51, C52, C53, C54, C55, C56, C57, C58, C59, C60, C61, C62, C63, C64, C65, C66, C67, C68, C69, C70, C71, C72, C73, C74, C75, C76, C77, C78, C79, C80, C81, C82, C83, C84, C85, C86, C87, C88, C89, C90, C91, C92, C93, C94, C95, C96, C97, C98, C99: 1nF_Ceramic, Capacitor_THT:C_Disc_D5.0mm_W2.5mm_P2.50mm, symbol PCM_SL_Capacitors:1nF_Ceramic
- removed R122, R123, R124, R125, R134, R135, R136, R137, R15, R16, R18, R19, R2, R20, R21, R22, R23, R24, R25, R26, R27, R28, R29, R30, R31, R32, R33, R34, R35, R36, R37, R38, R39, R40, R41, R42, R43, R44, R45, R46, R47, R48, R49, R50, R51, R52, R53, R54, R55, R56, R57, R58, R59, R60, R61, R62, R63, R64, R65, R66, R67, R68, R69, R70, R71, R72, R73, R74, R75, R76, R77, R78, R79, R80, R81, R82, R83, R84, R85, R86, R87, R88, R89, R90, R91, R92, R93, R94, R95, R96, R97: 10k, Resistor_THT:R_Axial_DIN0207_L6.3mm_D2.5mm_P10.16mm_Horizontal, symbol PCM_SL_Resistors:10k
Connections:
- net GND: now also SW4.1; no longer SW4.2, U6.20 (VCC)
- net VCC: now also U6.20 (VCC)
- net at D105.2 (A), D194.2 (A): now also SW4.2; no longer SW4.1

Commit message: Begun work on compiler, continued keyboard
Parts:
- removed U1, U4: 74LS08, Package_DIP:DIP-14_W7.62mm_Socket, symbol 74xx:74LS08
- removed unit 1 of U10
- removed U13, U14: 74LS30, Package_DIP:DIP-14_W7.62mm_Socket, symbol 74xx:74LS30
- removed Y1: ACO-1MHz-A, Oscillator:Oscillator_DIP-14, symbol Oscillator:ACO-xxxMHz-A
- added U1, U13, U4: 4068, Package_DIP:DIP-14_W7.62mm_Socket, symbol 4xxx_IEEE:4068
- added U14: 74LS240, Package_DIP:DIP-20_W7.62mm_Socket, symbol 74xx:74LS240
Connections:
- net ADJ_C15 is gone; now on net BUF-C0: R98.1, U2.4 (I7), U5.2 (A0)
- net ADJ_C8 is gone; now on net BUF-C1: R105.1, U2.10 (IO), U5.9 (A7)
- net ADJ_C9 is gone; now on net BUF-C2: R104.1, U2.11 (I1), U5.8 (A6)
- net BUF-C3 is gone; now on net BUF-C10: R110.1, U6.6 (A4), U7.13 (I3)
- net BUF-C4 is gone; now on net BUF-C11: R109.1, U6.5 (A3), U7.1 (I4)
- net BUF-C5 is gone; now on net BUF-C12: R108.1, U6.4 (A2), U7.2 (I5)
- net BUF-C6 is gone; now on net BUF-C13: R107.1, U6.3 (A1), U7.3 (I6)
- net BUF-C7 is gone; now on net BUF-C14: R106.1, U6.2 (A0), U7.4 (I7)
- net BIT0: now also U14.18 (O0a); no longer U9.9 (S0)
- net BIT1: now also U14.16 (O1a); no longer U9.7 (S1)
- net BIT2: now also U14.14 (O2a); no longer U7.9 (S0)
- net BIT3: now also U14.12 (O3a); no longer U7.7 (S1)
- net BIT4: now also U14.9 (O0b); no longer U7.6 (S2)
- net BIT5: now also U14.7 (O1b); no longer U2.9 (S0)
- net BIT6: now also U14.5 (O2b); no longer U2.7 (S1)
- net BIT7: now also U14.3 (O3b); no longer U2.6 (S2)
- net BUF-C0: now also U1.12 (H), U4.2 (A)
- net BUF-C1: now also U1.11 (G), U4.12 (H)
- net BUF-C2: now also U1.10 (F), U4.11 (G)
- net GND: now also U1.7 (Vss), U13.7 (Vss), U14.1 (OEa), U14.10 (GND), U14.19 (OEb), U4.7 (Vss)
- net VCC: now also U1.14 (Vdd), U13.10 (F), U13.11 (G), U13.12 (H), U13.14 (Vdd), U14.20 (VCC), U4.14 (Vdd)
- net at R120.1, U15.2, U8.1 (J)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: now also U8.12 (C)
- net at U8.9 (C): now also R121.1, U15.8, U8.11 (K), U8.8 (J); no longer U8.12 (C)
- net at U2.5 (EI): now also U4.1 (K)
- net at R118.1, U11.8 (A6), U9.11 (I1): now also U13.3 (B)
- net at R115.1, U11.5 (A3), U9.1 (I4): now also U13.9 (E)
- net at R119.1, U11.9 (A7), U9.10 (IO): now also U13.2 (A)
- net at R117.1, U11.7 (A5), U9.12 (I2): now also U13.4 (C)
- net at R116.1, U11.6 (A4), U9.13 (I3): now also U13.5 (D)
- net at U9.5 (EI): now also U13.1 (K)
- net at U7.5 (EI): now also U1.1 (K)
- net ADJ_C10 renamed BUF-C10
- net BUF-C10: now also U1.9 (E), U4.10 (F)
- net ADJ_C11 renamed BUF-C11
- net BUF-C11: now also U1.5 (D), U4.9 (E)
- net ADJ_C12 renamed BUF-C12
- net BUF-C12: now also U1.4 (C), U4.5 (D)
- net ADJ_C13 renamed BUF-C13
- net BUF-C13: now also U1.3 (B), U4.4 (C)
- net ADJ_C14 renamed BUF-C14
- net BUF-C14: now also U1.2 (A), U4.3 (B)
- new net: U14.4 (I1a), U9.7 (S1)
- new net: U14.2 (I0a), U9.9 (S0)
- new net: U14.11 (I0b), U7.6 (S2)
- new net: U14.8 (I3a), U7.7 (S1)
- new net: U14.6 (I2a), U7.9 (S0)
- new net: U14.13 (I1b), U2.9 (S0)
- new net: U14.15 (I2b), U2.7 (S1)
- new net: U14.17 (I3b), U2.6 (S2)
- no-connect marks 14 -> 16

Commit message: Continued
Parts:
- removed U10: 74LS30, Package_DIP:DIP-14_W7.62mm_Socket, symbol 74xx:74LS30
Changed lines of the file:
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@@
 	)
 	(label "GND"
-		(at 298.45 228.6 0)
-		(effects
-			(font
-				(size 1.27 1.27)
-			)
-			(justify left bottom)
-		)
-	)
-	(label "GND"
 		(at 116.84 64.77 180)
 		(effects
@@
 		)
 	)
-	(label "VCC"
-		(at 273.05 228.6 180)
-		(effects
-			(font
-				(size 1.27 1.27)
-			)
-			(justify right bottom)
-		)
-	)
 	(label "BUF-C2"
 		(at 502.92 171.45 180)
@@
 				)
 			)
-		)
-	)
-	(symbol
-		(lib_id "74xx:74LS30")
-		(at 285.75 228.6 90)
-		(unit 2)
-		(body_style 1)
-		(exclude_from_sim no)
-		(in_bom yes)
-		(on_board yes)
-		(in_pos_files yes)
-		(dnp no)
-		(fields_autoplaced yes)
-		(property "Reference" "U10"
-			(at 285.75 218.44 90)
-			(show_name no)
-			(do_not_autoplace no)
-			(effects
-				(font
-					(size 1.27 1.27)
-				)
-			)
-		)
-		(property "Value" "74LS30"
-			(at 285.75 220.98 90)
-			(show_name no)
-			(do_not_autoplace no)
-			(effects
-				(font
-					(size 1.27 1.27)
-				)
-			)
-		)
-		(property "Footprint" "Package_DIP:DIP-14_W7.62mm_Socket"
-			(at 285.75 228.6 0)
-			(hide yes)
-			(show_name no)
-			(do_not_autoplace no)
-			(effects
-				(font
-					(size 1.27 1.27)
-				)
-			)
-		)
-		(property "Datasheet" "http://www.ti.com/lit/gpn/sn74LS30"
-			(at 285.75 228.6 0)
-			(hide yes)
-			(show_name no)
-			(do_not_autoplace no)
-			(effects
-				(font
-					(size 1.27 1.27)
-				)
-			)
-		)
-		(property "Description" "8-input NAND"
-			(at 285.75 228.6 0)
-			(hide yes)
-			(show_name no)
-			(do_not_autoplace no)
-			(effects
-				(font
-					(size 1.27 1.27)
-				)
-			)
-		)
-		(pin "4"
-		)
-		(pin "11"
-		)
-		(pin "3"
-		)
-		(pin "5"
-		)
-		(pin "12"
-		)
-		(pin "7"
-		)
-		(pin "2"
-		)
-		(pin "1"
-		)
-		(pin "6"
-		)
-		(pin "8"
-		)
-		(pin "14"
-		)
-		(instances
-			(project "CYKEYBOARD"
-				(path "/eec78492-9332-4d17-adc9-870aaa031419"
-					(reference "U10")
-					(unit 2)
-				)
-			)

Commit message: Continued
Parts:
- removed R138, R140: 2.2k, Resistor_THT:R_Axial_DIN0207_L6.3mm_D2.5mm_P10.16mm_Horizontal, symbol PCM_SL_Resistors:2.2k
Connections:
- net VCC: now also U8.1 (J), U8.10 (~{R}), U8.11 (K), U8.13 (~{R}), U8.4 (K), U8.8 (J)
- net at R120.1, U15.2, U8.12 (C): no longer U8.1 (J), U8.4 (K)
- net at R121.1, U15.8, U8.9 (C): no longer U8.11 (K), U8.8 (J)
