File: Computer Designs/CYKEYBOARD/CYKEYBOARD.kicad_pcb (KiCad board)
At the start: 4 copper layers, 528.3 x 165.1 mm, 543 parts, among them J1 Conn_01x12, J2 Conn_01x03, J3 Conn_01x03, J4 Conn_01x09, K0 RESET, K13 READY, K14 ~~,,,,,,`, K15 !,,,,,,1, K16 @,,,,,,2, K17 #,,,,,,3, K18 $,,,,,,4, K19 %,,,,,,5, K20 ^,,,,,,6, K21 &,,,,,,7, K22 *,,,,,,8, K23 (,,,,,,9, K24 ),,,,,,0, K25 _,,,,,,-, K26 +,,,,,,=, K27 BACKSPACE, K28 INS, K29 HOME, K30 !,,,,,,1, K31 SAVE,,,,,,LOAD, K32 Q, K33 W, K34 E, K35 R, K36 T, K37 Y, K38 U, K39 I, K40 O, K41 P, K42 {,,,,,,[, K43 },,,,,,], K44 |,,,,,,\, K45 DEL, K46 HOLD, K47 @,,,,,,2, K48 SHIFT,,,,,,LOCK, K49 A, K50 S, K51 D, K52 F, K53 G, K54 H, K55 J, K56 K, K57 L, K58 :,,,,,,;, K59 ",,,,,,', K60 ENTER, K61 SHIFT, K62 Z, K63 X, K64 C, K65 V, K66 B, K67 N, K68 M, K69 <,,,,,,,, K70 >,,,,,,., K71 ?,,,,,,/, K72 SHIFT, K73 ^, K74 CTRL, K75 CYKA,,,,,,TECH, K76 ALT, K77 Blank, K78 ALT, K79 FN, K80 SELECT, K81 CTRL, K82 <, K83 \/, K84 >, K85 #,,,,,,3, K86 $,,,,,,4, K87 BACKSPACE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

Commit message: Continued
Parts:
- added D203: D, Diode_THT:D_T-1_P5.08mm_Horizontal, B.Cu at (392.1, 54.3)
- added D204: D, Diode_THT:D_T-1_P5.08mm_Horizontal, B.Cu at (414.6, 63.7)
- added D205: D, Diode_THT:D_T-1_P5.08mm_Horizontal, B.Cu at (397.6, 71.4)
- added D206: D, Diode_THT:D_T-1_P5.08mm_Horizontal, B.Cu at (405.5, 79.0)
- added D207: D, Diode_THT:D_T-1_P5.08mm_Horizontal, B.Cu at (424.5, 76.4)
- added D208: D, Diode_THT:D_T-1_P5.08mm_Horizontal, B.Cu at (392.1, 57.5)
- added D209: D, Diode_THT:D_T-1_P5.08mm_Horizontal, B.Cu at (415.6, 56.2)
- added D210: D, Diode_THT:D_T-1_P5.08mm_Horizontal, B.Cu at (411.5, 63.7)
- added D211: D, Diode_THT:D_T-1_P5.08mm_Horizontal, B.Cu at (419.4, 71.4)
- added D212: D, Diode_THT:D_T-1_P5.08mm_Horizontal, B.Cu at (421.0, 78.9)
- added D213: D, Diode_THT:D_T-1_P5.08mm_Horizontal, B.Cu at (424.6, 60.8)
- added D214: D, Diode_THT:D_T-1_P5.08mm_Horizontal, B.Cu at (403.1, 56.2)
- added D215: D, Diode_THT:D_T-1_P5.08mm_Horizontal, B.Cu at (417.7, 63.7)
- added D216: D, Diode_THT:D_T-1_P5.08mm_Horizontal, B.Cu at (413.2, 71.4)
- added D217: D, Diode_THT:D_T-1_P5.08mm_Horizontal, B.Cu at (408.6, 79.0)
- added D218: D, Diode_THT:D_T-1_P5.08mm_Horizontal, B.Cu at (424.5, 67.1)
- added D219: D, Diode_THT:D_T-1_P5.08mm_Horizontal, B.Cu at (406.2, 56.2)
- added D220: D, Diode_THT:D_T-1_P5.08mm_Horizontal, B.Cu at (396.0, 63.8)
- added D221: D, Diode_THT:D_T-1_P5.08mm_Horizontal, B.Cu at (400.7, 71.4)
- added D222: D, Diode_THT:D_T-1_P5.08mm_Horizontal, B.Cu at (399.3, 79.1)
- added D223: D, Diode_THT:D_T-1_P5.08mm_Horizontal, B.Cu at (424.6, 57.6)
- added D224: D, Diode_THT:D_T-1_P5.08mm_Horizontal, B.Cu at (399.8, 51.2)
- added D225: D, Diode_THT:D_T-1_P5.08mm_Horizontal, B.Cu at (405.3, 63.7)
- added D226: D, Diode_THT:D_T-1_P5.08mm_Horizontal, B.Cu at (407.0, 71.4)
- added D227: D, Diode_THT:D_T-1_P5.08mm_Horizontal, B.Cu at (411.7, 79.0)
- added D228: D, Diode_THT:D_T-1_P5.08mm_Horizontal, B.Cu at (424.5, 73.3)
- added D229: D, Diode_THT:D_T-1_P5.08mm_Horizontal, B.Cu at (412.5, 56.2)
- added D230: D, Diode_THT:D_T-1_P5.08mm_Horizontal, B.Cu at (399.1, 63.8)
- added D231: D, Diode_THT:D_T-1_P5.08mm_Horizontal, B.Cu at (416.3, 71.4)
- added D232: D, Diode_THT:D_T-1_P5.08mm_Horizontal, B.Cu at (417.9, 79.0)
- added D233: D, Diode_THT:D_T-1_P5.08mm_Horizontal, B.Cu at (402.2, 63.8)
- added D234: D, Diode_THT:D_T-1_P5.08mm_Horizontal, B.Cu at (403.8, 71.4)
- added D235: D, Diode_THT:D_T-1_P5.08mm_Horizontal, B.Cu at (402.4, 79.1)
- added D236: D, Diode_THT:D_T-1_P5.08mm_Horizontal, B.Cu at (424.6, 63.9)
- added D237: D, Diode_THT:D_T-1_P5.08mm_Horizontal, B.Cu at (409.4, 56.2)
- added D238: D, Diode_THT:D_T-1_P5.08mm_Horizontal, B.Cu at (408.4, 63.7)
- added D239: D, Diode_THT:D_T-1_P5.08mm_Horizontal, B.Cu at (410.1, 71.4)
- added D240: D, Diode_THT:D_T-1_P5.08mm_Horizontal, B.Cu at (414.8, 79.0)
- added D241: D, Diode_THT:D_T-1_P5.08mm_Horizontal, B.Cu at (424.6, 70.2)
- D1, D2, D3, D4, D5, D6, D7, D8: value D_Generic -> D; moved to B.Cu
- D100, D101, D102, D103, D104, D105, D106, D107, D108, D109, D110, D111, D112, D132, D133, D134, D135, D136, D137, D138, D139, D140, D141, D142, D143, D144, D145, D146, D147, D148, D149, D150, D151, D152, D153, D154, D155, D156, D157, D158, D159, D160, D161, D162, D163, D164, D165, D166, D167, D168, D169, D170, D171, D172, D173, D174, D175, D176, D177, D178, D179, D180, D181, D182, D183, D184, D186, D187, D188, D189, D190, D191, D192, D193, D195, D196, D197, D198, D201, D202, D30, D47, D86, D88, D89, D91, D98, D99, R120, R121, R138, R139, R140, R141, R3, R4, R5: moved to B.Cu
- moved D99 382.9 mm to (50.0, 163.6), turned to 90 degrees
- moved D103 365.3 mm to (74.0, 163.5), turned to 90 degrees
- moved D187 344.4 mm to (424.0, 82.6), turned to -90 degrees
- moved D186 344.3 mm to (424.5, 79.5)
- moved D102 341.5 mm to (98.0, 163.1), turned to 90 degrees
- moved D185 341.3 mm to (384.4, 51.2), turned to 180 degrees
- moved D188 338.7 mm to (394.5, 71.4), turned to -90 degrees
- moved D108 336.7 mm to (471.1, 35.1), turned to 90 degrees
- moved D198 335.5 mm to (392.1, 51.2), turned to 180 degrees
- moved D183 330.4 mm to (57.5, 144.6), turned to 90 degrees
- moved D197 327.2 mm to (399.7, 60.5), turned to 180 degrees
- moved D196 326.8 mm to (399.7, 57.5), turned to 180 degrees
- moved D195 326.4 mm to (399.7, 54.4), turned to 180 degrees
- moved D107 320.8 mm to (471.5, 53.1), turned to 90 degrees
- moved D194 316.5 mm to (384.4, 54.3), turned to 180 degrees
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Connections:
- D185 pad 1: Net-(D185-K) -> /FB0
- D194 pad 1: Net-(D185-K) -> /FB0
- D195 pad 1: Net-(D185-K) -> /FB2
- D196 pad 1: Net-(D185-K) -> /FB2
- D197 pad 1: Net-(D185-K) -> /FB2
- D198 pad 1: Net-(D185-K) -> /FB1
- D199 pad 1: Net-(D185-K) -> /FB0
- D200 pad 1: Net-(D185-K) -> /FB0
- D74 pad 1: /Row_0 -> /Row_5
- D75 pad 1: /Row_0 -> /Row_5
- D76 pad 1: /Row_0 -> /Row_5
- D77 pad 1: /Row_0 -> /Row_5
- D78 pad 1: /Row_0 -> /Row_5
- D81 pad 1: /Row_0 -> /Row_5
- J4 pad 1: /FB0 -> unconnected-(J4-Pin_1-Pad1)
- J4 pad 2: /FB1 -> /FB7
- J4 pad 3: /FB2 -> /FB6
- J4 pad 4: /FB3 -> /FB5
- J4 pad 6: /FB5 -> /FB3
- J4 pad 7: /FB6 -> /FB2
- J4 pad 8: /FB7 -> /FB1
- J4 pad 9: unconnected-(J4-Pin_9-Pad9) -> /FB0
Routing:
- net /Row_5: track 0.00 -> 877.3 mm
- net /Row_1: track 0.00 -> 784.9 mm
- net /Row_4: track 0.00 -> 565.2 mm, vias 0 -> 15
- net /Col_0: track 0.00 -> 556.2 mm, vias 0 -> 5
- net /Row_2: track 0.00 -> 537.7 mm, vias 0 -> 4
- net /Col_3: track 0.00 -> 514.5 mm, vias 0 -> 2
- net /Col_13: track 0.00 -> 508.7 mm, vias 0 -> 3
- net /Col_1: track 0.00 -> 379.1 mm, vias 0 -> 4
- net /Row_3: track 0.00 -> 376.1 mm, vias 0 -> 6
- net Net-(D107-K): track 0.00 -> 359.2 mm, vias 0 -> 5
- net Net-(D106-K): track 0.00 -> 341.6 mm, vias 0 -> 1
- net /Col_15: track 0.00 -> 337.4 mm
- net Net-(D200-A): track 0.00 -> 326.1 mm, vias 0 -> 3
- net /Col_8: track 0.00 -> 320.3 mm, vias 0 -> 1
- net /Col_5: track 0.00 -> 296.2 mm, vias 0 -> 10
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Other:
- board text added: "IRQ"

Commit message: Continued
Parts:
- K28: value INS -> HOME
- K29: value HOME -> MON
- K46: value HOLD -> BAS
- K94: value READY -> PAUSE
Changed lines of the file:
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@@
 			)
 		)
-		(property "Value" "HOLD"
+		(property "Value" "BAS"
 			(at -2.54 12.954 0)
 			(layer "F.SilkS")
@@
 			)
 		)
-		(property "Value" "READY"
+		(property "Value" "PAUSE"
 			(at -2.54 12.954 0)
 			(layer "F.Fab")
@@
 			)
 		)
-		(property "Value" "HOME"
+		(property "Value" "MON"
 			(at -2.54 12.954 0)
 			(layer "F.SilkS")
@@
 			)
 		)
-		(property "Value" "INS"
+		(property "Value" "HOME"
 			(at -2.54 12.954 0)
 			(layer "F.SilkS")

Commit message: Continued
Routing:
- net /GND: track 4014.3 -> 2662.9 mm
- net /Col_9: track 68.5 -> 941.8 mm, vias 0 -> 43
- net /Col_2: track 151.8 -> 745.4 mm, vias 5 -> 67
- net /Row_5: track 877.3 -> 1403.5 mm, vias 0 -> 24
- net /Col_10: track 68.3 -> 586.9 mm, vias 0 -> 37
- net /Col_3: track 514.5 -> 1030.9 mm, vias 2 -> 64
- net /Col_0: track 556.2 -> 1015.2 mm, vias 5 -> 50
- net /SHIFT_LOCK: track 9.36 -> 455.8 mm, vias 0 -> 1
- net /Col_14: track 288.3 -> 698.3 mm, vias 0 -> 16
- net /Col_7: track 227.5 -> 601.6 mm, vias 1 -> 50
- net Net-(D107-K): track 359.2 -> 0.00 mm, vias 5 -> 0
- net Net-(D106-K): track 341.6 -> 0.00 mm, vias 1 -> 0
- net /Col_8: track 320.3 -> 653.1 mm, vias 1 -> 49
- net /Col_4: track 116.0 -> 444.1 mm, vias 4 -> 21
- net /Col_13: track 508.7 -> 835.5 mm, vias 3 -> 20
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