File: Computer Designs/CYKEYBOARD/CYKEYBOARD.kicad_pcb (KiCad board)
At the start: 6 copper layers, 528.3 x 165.1 mm, 507 parts, among them J1 Conn_01x12, J2 Conn_01x03, J3 Conn_01x03, K0 RESET, K13 READY, K14 ~~,,,,,,`, K15 !,,,,,,1, K16 @,,,,,,2, K17 #,,,,,,3, K18 $,,,,,,4, K19 %,,,,,,5, K20 ^,,,,,,6, K21 &,,,,,,7, K22 *,,,,,,8, K23 (,,,,,,9, K24 ),,,,,,0, K25 _,,,,,,-, K26 +,,,,,,=, K27 BACKSPACE, K28 HOME, K29 MON, K30 !,,,,,,1, K31 SAVE,,,,,,LOAD, K32 Q, K33 W, K34 E, K35 R, K36 T, K37 Y, K38 U, K39 I, K40 O, K41 P, K42 {,,,,,,[, K43 },,,,,,], K44 |,,,,,,\, K45 DEL, K46 BAS, K47 @,,,,,,2, K48 SHIFT,,,,,,LOCK, K49 A, K50 S, K51 D, K52 F, K53 G, K54 H, K55 J, K56 K, K57 L, K58 :,,,,,,;, K59 ",,,,,,', K60 ENTER, K61 SHIFT, K62 Z, K63 X, K64 C, K65 V, K66 B, K67 N, K68 M, K69 <,,,,,,,, K70 >,,,,,,., K71 ?,,,,,,/, K72 SHIFT, K73 ^, K74 CTRL, K75 CYKA,,,,,,TECH, K76 ALT, K77 Blank, K78 ALT, K79 FN, K80 SELECT, K81 CTRL, K82 <, K83 \/, K84 >, K85 #,,,,,,3, K86 $,,,,,,4, K87 BACKSPACE, K88 ),,,,,,0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

Commit message: Continued
Other:
- copper layers 6 -> 2
Changed lines of the file:
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@@
 	(layers
 		(0 "F.Cu" jumper)
-		(4 "In1.Cu" mixed)
-		(6 "In2.Cu" signal)
-		(8 "In3.Cu" signal)
-		(10 "In4.Cu" signal)
 		(2 "B.Cu" signal)
 		(9 "F.Adhes" user "F.Adhesive")
@@
 			)
 			(layer "dielectric 1"
-				(type "prepreg")
-				(thickness 0.1)
-				(material "FR4")
-				(epsilon_r 4.5)
-				(loss_tangent 0.02)
-			)
-			(layer "In1.Cu"
-				(type "copper")
-				(thickness 0.035)
-			)
-			(layer "dielectric 2"
 				(type "core")
-				(thickness 0.535)
-				(material "FR4")
-				(epsilon_r 4.5)
-				(loss_tangent 0.02)
-			)
-			(layer "In2.Cu"
-				(type "copper")
-				(thickness 0.035)
-			)
-			(layer "dielectric 3"
-				(type "prepreg")
-				(thickness 0.1)
-				(material "FR4")
-				(epsilon_r 4.5)
-				(loss_tangent 0.02)
-			)
-			(layer "In3.Cu"
-				(type "copper")
-				(thickness 0.035)
-			)
-			(layer "dielectric 4"
-				(type "core")
-				(thickness 0.535)
-				(material "FR4")
-				(epsilon_r 4.5)
-				(loss_tangent 0.02)
-			)
-			(layer "In4.Cu"
-				(type "copper")
-				(thickness 0.035)
-			)
-			(layer "dielectric 5"
-				(type "prepreg")
-				(thickness 0.1)
+				(thickness 1.51)
 				(material "FR4")
 				(epsilon_r 4.5)
@@
 		(capping no)
 		(filling no)
+		(zone_defaults)
 		(pcbplotparams
 			(layerselection 0x00000000_00000000_5555555f_ffffffff)

Commit message: Continued
Parts:
- added D185: D, Diode_THT:D_T-1_P5.08mm_Horizontal, B.Cu at (526.4, 159.8)
- added D188: D, Diode_THT:D_T-1_P5.08mm_Horizontal, B.Cu at (489.7, 158.4)
- added D189: D, Diode_THT:D_T-1_P5.08mm_Horizontal, B.Cu at (526.3, 115.4)
- added D190: D, Diode_THT:D_T-1_P5.08mm_Horizontal, B.Cu at (488.1, 115.6)
- added D191: D, Diode_THT:D_T-1_P5.08mm_Horizontal, B.Cu at (488.1, 39.8)
- added D192: D, Diode_THT:D_T-1_P5.08mm_Horizontal, B.Cu at (526.1, 39.9)
- added D193: D, Diode_THT:D_T-1_P5.08mm_Horizontal, B.Cu at (488.1, 78.0)
- added D194: D, Diode_THT:D_T-1_P5.08mm_Horizontal, B.Cu at (526.2, 76.9)
- added Q1: 2N2222A-TO92, PCM_Package_TO_SOT_THT_AKL:TO-92_Inline_Wide_EBC, B.Cu at (182.5, 28.8)
- added Q2: 2N2222A-TO92, PCM_Package_TO_SOT_THT_AKL:TO-92_Inline_Wide_EBC, B.Cu at (193.9, 28.8)
- added R7: 3.3k, Resistor_THT:R_Axial_DIN0207_L6.3mm_D2.5mm_P10.16mm_Horizontal, B.Cu at (313.3, 56.6)
- added U1: 74LS08, Package_DIP:DIP-14_W7.62mm_Socket, B.Cu at (110.2, 38.3)
- added U10: 74LS30, Package_DIP:DIP-14_W7.62mm_Socket_LongPads, B.Cu at (401.5, 58.0)
- added U11: 74AHC541, Package_DIP:DIP-20_W7.62mm_Socket, B.Cu at (449.8, 24.4)
- added U12: 74HC00, Package_DIP:DIP-14_W7.62mm_Socket, B.Cu at (424.5, 57.8)
- added U13: 74LS30, Package_DIP:DIP-14_W7.62mm_Socket_LongPads, B.Cu at (446.5, 57.8)
- added U14: 74LS30, Package_DIP:DIP-14_W7.62mm_Socket_LongPads, B.Cu at (263.0, 33.5)
- added U15: 74HC14, Package_DIP:DIP-14_W7.62mm_Socket_LongPads, B.Cu at (66.0, 38.5)
- added U4: 74LS08, Package_DIP:DIP-14_W7.62mm_Socket, B.Cu at (89.5, 38.3)
- added U5: 74AHC541, Package_DIP:DIP-20_W7.62mm_Socket, B.Cu at (404.5, 24.5)
- added U6: 74AHC541, Package_DIP:DIP-20_W7.62mm_Socket, B.Cu at (426.4, 24.5)
- moved U3 136.9 mm to (239.0, 33.9)
- moved D186 98.9 mm to (328.0, 58.0)
- moved D187 98.0 mm to (328.1, 62.3), turned to 0 degrees
- moved C102 40.9 mm to (511.0, 102.7)
- moved D110 40.9 mm to (509.1, 114.8)
- moved SW6 40.9 mm to (520.2, 106.0)
- moved R135 40.9 mm to (526.2, 102.7)
- moved C99 40.7 mm to (510.5, 27.3)
- moved D107 40.7 mm to (509.6, 38.8)
- moved R124 40.7 mm to (525.7, 27.3)
- moved SW2 40.7 mm to (520.1, 30.3)
- moved SW4 40.6 mm to (520.2, 68.9)
- moved D105 40.6 mm to (509.7, 76.4)
- moved R122 40.6 mm to (526.0, 65.8)
- moved C97 40.6 mm to (510.7, 65.9)
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Connections:
- D1 pad 2: /GS1 -> Net-(D1-A)
- D112 pad 1: unconnected-(D112-K-Pad1) -> /Col_11
- D2 pad 2: /GS2 -> Net-(D2-A)
- D3 pad 2: /GS3 -> Net-(D3-A)
- J3 pad 2: unconnected-(J3-Pin_2-Pad2) -> Net-(J3-Pin_2)
- R100 pad 1: /Col_13 -> /ADJ_C13
- R101 pad 1: /Col_12 -> /ADJ_C12
- R102 pad 1: /Col_11 -> /ADJ_C11
- R103 pad 1: /Col_10 -> /ADJ_C10
- R104 pad 1: /Col_9 -> /ADJ_C9
- R105 pad 1: /Col_8 -> /ADJ_C8
- R106 pad 1: /Col_7 -> /BUF-C7
- R107 pad 1: /Col_6 -> /BUF-C6
- R108 pad 1: /Col_5 -> /BUF-C5
- R109 pad 1: /Col_4 -> /BUF-C4
- R110 pad 1: /Col_3 -> /BUF-C3
- R111 pad 1: /Col_2 -> /BUF-C2
- R112 pad 1: /Col_1 -> /BUF-C1
- R113 pad 1: /Col_0 -> /BUF-C0
- R115 pad 1: /Row_5 -> Net-(U11-A3)
- R116 pad 1: /Row_4 -> Net-(U11-A4)
- R117 pad 1: /Row_3 -> Net-(U11-A5)
- R118 pad 1: /Row_2 -> Net-(U11-A6)
- R119 pad 1: /Row_1 -> Net-(U11-A7)
- R3 pad 1: /GND -> /VCC
- R98 pad 1: /Col_15 -> /ADJ_C15
- R99 pad 1: /Col_14 -> /ADJ_C14
- SW4 pad 1: /GND -> Net-(D105-A)
- SW4 pad 2: Net-(D105-A) -> /GND
- U2 pad 1: unconnected-(U2-I4-Pad1) -> /ADJ_C12
- U2 pad 10: unconnected-(U2-IO-Pad10) -> /ADJ_C8
- U2 pad 11: unconnected-(U2-I1-Pad11) -> /ADJ_C9
- U2 pad 12: unconnected-(U2-I2-Pad12) -> /ADJ_C10
- U2 pad 13: unconnected-(U2-I3-Pad13) -> /ADJ_C11
- U2 pad 15: unconnected-(U2-EO-Pad15) -> /EO0
- U2 pad 2: unconnected-(U2-I5-Pad2) -> /ADJ_C13
- U2 pad 3: unconnected-(U2-I6-Pad3) -> /ADJ_C14
- U2 pad 4: unconnected-(U2-I7-Pad4) -> /ADJ_C15
- U2 pad 5: /GND -> Net-(U2-EI)
- U2 pad 6: unconnected-(U2-S2-Pad6) -> /BIT7
- U2 pad 7: unconnected-(U2-S1-Pad7) -> /BIT6
- U2 pad 9: unconnected-(U2-S0-Pad9) -> /BIT5
- U7 pad 1: unconnected-(U7-I4-Pad1) -> /BUF-C4
- U7 pad 10: unconnected-(U7-IO-Pad10) -> /BUF-C0
- U7 pad 11: unconnected-(U7-I1-Pad11) -> /BUF-C1
- U7 pad 12: unconnected-(U7-I2-Pad12) -> /BUF-C2
- U7 pad 13: unconnected-(U7-I3-Pad13) -> /BUF-C3
- U7 pad 15: unconnected-(U7-EO-Pad15) -> /EO1
- U7 pad 2: unconnected-(U7-I5-Pad2) -> /BUF-C5
- U7 pad 3: unconnected-(U7-I6-Pad3) -> /BUF-C6
- U7 pad 4: unconnected-(U7-I7-Pad4) -> /BUF-C7
- U7 pad 5: /GND -> Net-(U7-EI)
- U7 pad 6: unconnected-(U7-S2-Pad6) -> /BIT4
- U7 pad 7: unconnected-(U7-S1-Pad7) -> /BIT3
- U7 pad 9: unconnected-(U7-S0-Pad9) -> /BIT2
- U9 pad 1: unconnected-(U9-I4-Pad1) -> Net-(U11-A3)
- U9 pad 10: unconnected-(U9-IO-Pad10) -> Net-(U11-A7)
- U9 pad 11: unconnected-(U9-I1-Pad11) -> Net-(U11-A6)
- U9 pad 12: unconnected-(U9-I2-Pad12) -> Net-(U11-A5)
- U9 pad 13: unconnected-(U9-I3-Pad13) -> Net-(U11-A4)
- U9 pad 15: unconnected-(U9-EO-Pad15) -> /EO2
- U9 pad 5: /GND -> Net-(U9-EI)
- U9 pad 7: unconnected-(U9-S1-Pad7) -> /BIT1
- U9 pad 9: unconnected-(U9-S0-Pad9) -> /BIT0
Routing:
- net /GND: track 0.00 -> 2228.9 mm
- net Net-(D111-A): track 0.00 -> 27.3 mm
- net Net-(D112-A): track 0.00 -> 26.4 mm
- net Net-(D108-A): track 0.00 -> 25.5 mm
- net Net-(D110-A): track 0.00 -> 25.4 mm
- net Net-(D106-A): track 0.00 -> 25.2 mm
- net Net-(D109-A): track 0.00 -> 25.1 mm
- net Net-(D147-A): track 0.00 -> 24.8 mm
- net Net-(D153-A): track 0.00 -> 24.8 mm
- net Net-(D170-A): track 0.00 -> 24.8 mm
- net Net-(D144-A): track 0.00 -> 24.8 mm
- net Net-(D129-A): track 0.00 -> 24.7 mm
- net Net-(D145-A): track 0.00 -> 24.7 mm
- net Net-(D169-A): track 0.00 -> 24.6 mm
- net Net-(D121-A): track 0.00 -> 24.6 mm
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
Commit message: Continued
Parts:
- removed C1, C100, C101, C102, C103, C104, C14, C15, C17, C18, C19, C20, C21, C22, C23, C24, C25, C26, C27, C28, C29, C30, C31, C32, C33, C34, C35, C36, C37, C38, C39, C40, C41, C42, C43, C44, C45, C46, C47, C48, C49, C50, C51, C52, C53, C54, C55, C56, C57, C58, C59, C60, C61, C62, C63, C64, C65, C66, C67, C68, C69, C70, C71, C72, C73, C74, C75, C76, C77, C78, C79, C80, C81, C82, C83, C84, C85, C86, C87, C88, C89, C90, C91, C92, C93, C94, C95, C96, C97, C98, C99: 1nF_Ceramic, Capacitor_THT:C_Disc_D5.0mm_W2.5mm_P2.50mm
- removed R122, R123, R124, R125, R134, R135, R136, R137, R15, R16, R18, R19, R2, R20, R21, R22, R23, R24, R25, R26, R27, R28, R29, R30, R31, R32, R33, R34, R35, R36, R37, R38, R39, R40, R41, R42, R43, R44, R45, R46, R47, R48, R49, R50, R51, R52, R53, R54, R55, R56, R57, R58, R59, R60, R61, R62, R63, R64, R65, R66, R67, R68, R69, R70, R71, R72, R73, R74, R75, R76, R77, R78, R79, R80, R81, R82, R83, R84, R85, R86, R87, R88, R89, R90, R91, R92, R93, R94, R95, R96, R97: 10k, Resistor_THT:R_Axial_DIN0207_L6.3mm_D2.5mm_P10.16mm_Horizontal
- U10, U13, U14, U15: footprint Package_DIP:DIP-14_W7.62mm_Socket_LongPads -> Package_DIP:DIP-14_W7.62mm_Socket
- moved D91 16.2 mm to (425.8, 125.4)
- moved D153 15.9 mm to (441.9, 125.6)
- moved D105 1.63 mm to (509.6, 78.0)
- moved D194 1.63 mm to (526.1, 78.5)
Connections:
- SW4 pad 1: Net-(D105-A) -> /GND
- SW4 pad 2: /GND -> Net-(D105-A)
- U6 pad 20: /GND -> /VCC
Routing:
- net /GND: track 2228.9 -> 4241.9 mm
- net /VCC: track 0.00 -> 634.7 mm
- net /Row_5: track 0.00 -> 625.2 mm
- net /Row_1: track 0.00 -> 476.6 mm
- net /Col_0: track 0.00 -> 258.3 mm, vias 0 -> 8
- net /Col_5: track 0.00 -> 69.9 mm, vias 0 -> 6
- net /Col_4: track 0.00 -> 69.6 mm, vias 0 -> 6
- net /Col_3: track 0.00 -> 69.4 mm, vias 0 -> 6
- net /Col_2: track 0.00 -> 69.2 mm, vias 0 -> 6
- net /Col_1: track 0.00 -> 69.1 mm, vias 0 -> 6
- net /IRQ: track 0.00 -> 57.7 mm
- net /RST: track 0.00 -> 22.6 mm
- net Net-(D157-A): track 0.00 -> 17.8 mm
- net Net-(D77-A): track 0.00 -> 17.4 mm
- net Net-(D155-A): track 0.00 -> 17.4 mm
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
Commit message: Continued
Routing:
- net /Col_13: track 0.00 -> 389.1 mm, vias 0 -> 7
- net /BUF-C1: track 0.00 -> 381.9 mm, vias 0 -> 13
- net /RDY_LOCK: track 0.00 -> 356.7 mm, vias 0 -> 8
- net /Col_15: track 0.00 -> 339.5 mm, vias 0 -> 6
- net /Row_4: track 0.00 -> 314.1 mm
- net Net-(J3-Pin_2): track 0.00 -> 293.1 mm, vias 0 -> 5
- net /Col_11: track 0.00 -> 286.4 mm, vias 0 -> 4
- net /Row_3: track 0.00 -> 280.9 mm, vias 0 -> 2
- net /ADJ_C15: track 0.00 -> 262.8 mm
- net /SHIFT_LED: track 0.00 -> 232.3 mm, vias 0 -> 2
- net /Col_12: track 0.00 -> 220.2 mm, vias 0 -> 5
- net /Col_6: track 0.00 -> 211.4 mm, vias 0 -> 8
- net /ADJ_C9: track 0.00 -> 207.5 mm, vias 0 -> 9
- net /SHIFT_LOCK: track 0.00 -> 187.2 mm
- net /Col_7: track 0.00 -> 175.2 mm, vias 0 -> 6
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
Commit message: Begun work on compiler, continued keyboard
Parts:
- removed U10: 74LS30, Package_DIP:DIP-14_W7.62mm_Socket
- removed Y1: ACO-1MHz-A, Oscillator:Oscillator_DIP-14
- U1, U4: value 74LS08 -> 4068
- U13: value 74LS30 -> 4068
- U14: value 74LS30 -> 74LS240; footprint Package_DIP:DIP-14_W7.62mm_Socket -> Package_DIP:DIP-20_W7.62mm_Socket
- moved U12 200.7 mm to (223.8, 55.1)
- moved U6 200.7 mm to (225.7, 21.8)
- moved U11 200.7 mm to (249.1, 21.8)
- moved U13 200.7 mm to (245.8, 55.2)
- moved U5 200.7 mm to (203.8, 21.8)
- moved J1 97.9 mm to (418.3, 28.7)
- moved U3 90.8 mm to (150.1, 52.4)
- moved Q2 85.0 mm to (110.0, 42.2)
- moved Q1 85.0 mm to (98.6, 42.2)
- moved U14 84.4 mm to (179.3, 44.1)
- moved R5 81.5 mm to (50.9, 28.6)
- moved U9 64.3 mm to (121.7, 49.6)
- moved U7 63.5 mm to (150.1, 27.8)
- moved R4 55.6 mm to (264.1, 31.5)
- moved R121 43.2 mm to (266.6, 56.2)
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Connections:
- R100 pad 1: /ADJ_C13 -> /BUF-C13
- R101 pad 1: /ADJ_C12 -> /BUF-C12
- R102 pad 1: /ADJ_C11 -> /BUF-C11
- R103 pad 1: /ADJ_C10 -> /BUF-C10
- R104 pad 1: /ADJ_C9 -> /BUF-C2
- R105 pad 1: /ADJ_C8 -> /BUF-C1
- R106 pad 1: /BUF-C7 -> /BUF-C14
- R107 pad 1: /BUF-C6 -> /BUF-C13
- R108 pad 1: /BUF-C5 -> /BUF-C12
- R109 pad 1: /BUF-C4 -> /BUF-C11
- R110 pad 1: /BUF-C3 -> /BUF-C10
- R120 pad 1: Net-(U8A-J) -> Net-(U8A-C)
- R121 pad 1: Net-(U8B-J) -> Net-(U8B-C)
- R98 pad 1: /ADJ_C15 -> /BUF-C0
- R99 pad 1: /ADJ_C14 -> /BUF-C14
- U1 pad 1: /BUF-C7 -> Net-(U1-K)
- U1 pad 10: /ADJ_C13 -> /BUF-C2
- U1 pad 11: /ADJ_C12 -> /BUF-C1
- U1 pad 12: /BUF-C4 -> /BUF-C0
- U1 pad 13: /ADJ_C12 -> unconnected-(U1-J-Pad13)
- U1 pad 2: /ADJ_C15 -> /BUF-C14
- U1 pad 3: /ADJ_C15 -> /BUF-C13
- U1 pad 4: /BUF-C6 -> /BUF-C12
- U1 pad 5: /ADJ_C14 -> /BUF-C11
- U1 pad 6: /ADJ_C14 -> unconnected-(U1-NC-Pad6)
- U1 pad 8: /ADJ_C13 -> unconnected-(U1-NC-Pad8)
- U1 pad 9: /BUF-C5 -> /BUF-C10
- U13 pad 1: /BUF-C7 -> Net-(U13-K)
- U13 pad 10: (no net) -> /VCC
- U13 pad 11: /BUF-C1 -> /VCC
- U13 pad 12: /BUF-C0 -> /VCC
- U13 pad 13: (no net) -> unconnected-(U13-J-Pad13)
- U13 pad 2: /BUF-C6 -> Net-(U11-A7)
- U13 pad 3: /BUF-C5 -> Net-(U11-A6)
- U13 pad 4: /BUF-C4 -> Net-(U11-A5)
- U13 pad 5: /BUF-C3 -> Net-(U11-A4)
- U13 pad 6: /BUF-C2 -> unconnected-(U13-NC-Pad6)
- U13 pad 8: Net-(U7-EI) -> unconnected-(U13-NC-Pad8)
- U13 pad 9: (no net) -> Net-(U11-A3)
- U14 pad 1: /ADJ_C15 -> /GND
- U14 pad 10: (no net) -> /GND
- U14 pad 11: /ADJ_C9 -> Net-(U14-I0b)
- U14 pad 12: /ADJ_C8 -> /BIT3
- U14 pad 13: (no net) -> Net-(U14-I1b)
- U14 pad 14: /VCC -> /BIT2
- U14 pad 2: /ADJ_C14 -> Net-(U14-I0a)
- U14 pad 3: /ADJ_C13 -> /BIT7
- U14 pad 4: /ADJ_C12 -> Net-(U14-I1a)
- U14 pad 5: /ADJ_C11 -> /BIT6
- U14 pad 6: /ADJ_C10 -> Net-(U14-I2a)
- U14 pad 7: /GND -> /BIT5
- U14 pad 8: Net-(U2-EI) -> Net-(U14-I3a)
- U14 pad 9: (no net) -> /BIT4
- U15 pad 2: Net-(U8A-J) -> Net-(U8A-C)
- U15 pad 8: Net-(U8B-J) -> Net-(U8B-C)
- U2 pad 1: /ADJ_C12 -> /BUF-C12
- U2 pad 10: /ADJ_C8 -> /BUF-C1
- U2 pad 11: /ADJ_C9 -> /BUF-C2
- U2 pad 12: /ADJ_C10 -> /BUF-C10
- U2 pad 13: /ADJ_C11 -> /BUF-C11
- U2 pad 2: /ADJ_C13 -> /BUF-C13
- U2 pad 3: /ADJ_C14 -> /BUF-C14
- U2 pad 4: /ADJ_C15 -> /BUF-C0
- U2 pad 6: /BIT7 -> Net-(U14-I3b)
- U2 pad 7: /BIT6 -> Net-(U14-I2b)
- U2 pad 9: /BIT5 -> Net-(U14-I1b)
- U4 pad 1: /BUF-C3 -> Net-(U2-EI)
- U4 pad 10: /ADJ_C9 -> /BUF-C10
- U4 pad 11: /ADJ_C8 -> /BUF-C2
- U4 pad 12: /BUF-C0 -> /BUF-C1
- U4 pad 13: /ADJ_C8 -> unconnected-(U4-J-Pad13)
- U4 pad 2: /ADJ_C11 -> /BUF-C0
- U4 pad 3: /ADJ_C11 -> /BUF-C14
- U4 pad 4: /BUF-C2 -> /BUF-C13
- U4 pad 5: /ADJ_C10 -> /BUF-C12
- U4 pad 6: /ADJ_C10 -> unconnected-(U4-NC-Pad6)
- U4 pad 8: /ADJ_C9 -> unconnected-(U4-NC-Pad8)
- U4 pad 9: /BUF-C1 -> /BUF-C11
- U5 pad 2: /ADJ_C15 -> /BUF-C0
- U5 pad 3: /ADJ_C14 -> /BUF-C14
- U5 pad 4: /ADJ_C13 -> /BUF-C13
- U5 pad 5: /ADJ_C12 -> /BUF-C12
- U5 pad 6: /ADJ_C11 -> /BUF-C11
- U5 pad 7: /ADJ_C10 -> /BUF-C10
- U5 pad 8: /ADJ_C9 -> /BUF-C2
- U5 pad 9: /ADJ_C8 -> /BUF-C1
- U6 pad 2: /BUF-C7 -> /BUF-C14
- U6 pad 3: /BUF-C6 -> /BUF-C13
- U6 pad 4: /BUF-C5 -> /BUF-C12
- U6 pad 5: /BUF-C4 -> /BUF-C11
- U6 pad 6: /BUF-C3 -> /BUF-C10
- U7 pad 1: /BUF-C4 -> /BUF-C11
- U7 pad 13: /BUF-C3 -> /BUF-C10
- U7 pad 2: /BUF-C5 -> /BUF-C12
- U7 pad 3: /BUF-C6 -> /BUF-C13
- U7 pad 4: /BUF-C7 -> /BUF-C14
- U7 pad 5: Net-(U7-EI) -> Net-(U1-K)
- U7 pad 6: /BIT4 -> Net-(U14-I0b)
- U7 pad 7: /BIT3 -> Net-(U14-I3a)
- U7 pad 9: /BIT2 -> Net-(U14-I2a)
- U8 pad 1: Net-(U8A-J) -> Net-(U8A-C)
- U8 pad 11: Net-(U8B-J) -> Net-(U8B-C)
- U8 pad 4: Net-(U8A-J) -> Net-(U8A-C)
- U8 pad 8: Net-(U8B-J) -> Net-(U8B-C)
- U8 pad 9: Net-(U8A-C) -> Net-(U8B-C)
- U9 pad 5: Net-(U9-EI) -> Net-(U13-K)
- U9 pad 7: /BIT1 -> Net-(U14-I1a)
- U9 pad 9: /BIT0 -> Net-(U14-I0a)
Routing:
- net /Col_14: track 20.3 -> 485.8 mm
- net /Col_15: track 339.5 -> 788.6 mm, vias 6 -> 8
- net /GND: track 4241.9 -> 3902.0 mm
- net /Col_5: track 69.9 -> 381.0 mm, vias 6 -> 8
- net /Col_0: track 258.3 -> 554.7 mm, vias 8 -> 15
- net /Row_5: track 625.2 -> 913.6 mm, vias 0 -> 15
- net /Col_7: track 175.2 -> 462.8 mm, vias 6 -> 9
- net /ADJ_C15: track 262.8 -> 0.00 mm
- net Net-(U8B-C): track 0.00 -> 247.3 mm, vias 0 -> 12
- net /Col_11: track 286.4 -> 44.3 mm, vias 4 -> 0
- net Net-(D201-A): track 0.00 -> 222.9 mm, vias 0 -> 9
- net Net-(U8B-~{R}): track 0.00 -> 207.7 mm, vias 0 -> 15
- net /ADJ_C9: track 207.5 -> 0.00 mm, vias 9 -> 0
- net Net-(U8A-~{R}): track 0.00 -> 194.8 mm, vias 0 -> 16
- net /VCC: track 787.5 -> 977.0 mm
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
Commit message: Continued
Routing:
- net /Row_3: track 293.3 -> 403.5 mm, vias 6 -> 14
Changed lines of the file:
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@@
+	)
+	(segment
+		(start 237.45 108.15)
+		(end 237.45 101)
+		(width 0.25)
+		(layer "F.Cu")
+		(net "/Row_3")
+	)
+	(segment
+		(start 233.7 96.25)
+		(end 233.7 81.4)
+		(width 0.25)
+		(layer "F.Cu")
+		(net "/Row_3")
+	)
+	(segment
+		(start 233.45 117.3)
+		(end 233.45 115.55)
+		(width 0.25)
+		(layer "F.Cu")
+		(net "/Row_3")
+	)
+	(segment
+		(start 235.45 98)
+		(end 233.7 96.25)
+		(width 0.25)
+		(layer "F.Cu")
+		(net "/Row_3")
+	)
+	(segment
+		(start 236.95 78.85)
+		(end 239.2 76.6)
+		(width 0.25)
+		(layer "F.Cu")
+		(net "/Row_3")
 	)
 	(segment
@@
 	)
 	(segment
+		(start 237.45 101)
+		(end 237.25 100.8)
+		(width 0.25)
+		(layer "F.Cu")
+		(net "/Row_3")
+	)
+	(segment
+		(start 239.2 76.6)
+		(end 251.5 76.6)
+		(width 0.25)
+		(layer "F.Cu")
+		(net "/Row_3")
+	)
+	(segment
+		(start 233.45 115.55)
+		(end 233.4 115.5)
+		(width 0.25)
+		(layer "F.Cu")
+		(net "/Row_3")
+	)
+	(segment
 		(start 291.9 146.15)
 		(end 291.05 145.3)
@@
 	)
 	(via
+		(at 233.45 117.3)
+		(size 0.25)
+		(drill 0.3)
+		(layers "F.Cu" "B.Cu")
+		(net "/Row_3")
+	)
+	(via
+		(at 233.4 115.5)
+		(size 0.25)
+		(drill 0.3)
+		(layers "F.Cu" "B.Cu")
+		(net "/Row_3")
+	)
+	(via
+		(at 236.95 78.85)
+		(size 0.25)
+		(drill 0.3)
+		(layers "F.Cu" "B.Cu")
+		(net "/Row_3")
+	)
+	(via
+		(at 251.5 76.6)
+		(size 0.25)
+		(drill 0.3)
+		(layers "F.Cu" "B.Cu")
+		(net "/Row_3")
+	)
+	(via
+		(at 233.7 81.4)
+		(size 0.25)
+		(drill 0.3)
+		(layers "F.Cu" "B.Cu")
+		(net "/Row_3")
+	)
+	(via
+		(at 235.45 98)
+		(size 0.25)
+		(drill 0.3)
+		(layers "F.Cu" "B.Cu")
+		(net "/Row_3")
+	)
+	(via
 		(at 291.3 133.75)
 		(size 0.25)
@@
 	)
 	(via
+		(at 237.25 100.8)
+		(size 0.25)
+		(drill 0.3)
+		(layers "F.Cu" "B.Cu")
+		(net "/Row_3")
+	)
+	(via
 		(at 291.05 139.1)
 		(size 0.25)
@@
 		(drill 0.3)
 		(layers "F.Cu" "B.Cu")
+		(net "/Row_3")
+	)
+	(via
+		(at 237.45 108.15)
+		(size 0.25)
+		(drill 0.3)
+		(layers "F.Cu" "B.Cu")
+		(net "/Row_3")
+	)
+	(segment
+		(start 232.0225 122.35222)
+		(end 233.45 120.92472)
+		(width 0.25)
+		(layer "B.Cu")
+		(net "/Row_3")
+	)
+	(segment
+		(start 237.25 100.8)
+		(end 237.25 99.8)
+		(width 0.25)
+		(layer "B.Cu")
 		(net "/Row_3")
 	)
@@
 	)
 	(segment
+		(start 247.7 46.25)
+		(end 248.05 46.6)
+		(width 0.25)
+		(layer "B.Cu")
+		(net "/Row_3")
+	)
+	(segment
+		(start 233.45 120.92472)
+		(end 233.45 117.3)
+		(width 0.25)
+		(layer "B.Cu")
+		(net "/Row_3")
+	)
+	(segment
+		(start 233.4 112.2)
+		(end 237.45 108.15)
+		(width 0.25)
+		(layer "B.Cu")
+		(net "/Row_3")
+	)
+	(segment
 		(start 291.05 136.65)
 		(end 291.3 136.4)
@@
 	)
 	(segment
+		(start 251.5 76.6)
+		(end 251.325 76.425)
+		(width 0.25)
+		(layer "B.Cu")
+		(net "/Row_3")
+	)
+	(segment
 		(start 61.7625 126.405)
 		(end 78.4325 126.405)
@@
 	)
 	(segment
+		(start 233.4 115.5)
+		(end 233.4 112.2)
+		(width 0.25)
+		(layer "B.Cu")
+		(net "/Row_3")
+	)
+	(segment
 		(start 285.635 163.315)
 		(end 292.25 156.7)
@@
 	)
 	(segment
+		(start 247.7 45.85)
+		(end 247.7 46.25)
+		(width 0.25)
+		(layer "B.Cu")
+		(net "/Row_3")
+	)
+	(segment
 		(start 193.9225 125.215)
 		(end 195.6125 126.905)
@@
 	)
 	(segment
+		(start 247.7 45.85)
+		(end 241.43 39.58)
+		(width 0.25)
+		(layer "B.Cu")
+		(net "/Row_3")
+	)
+	(segment
 		(start 230.4125 126.825)
 		(end 232.0225 125.215)
@@
 	)
 	(segment
+		(start 251.325 76.425)
+		(end 251.325 47.275)
+		(width 0.25)
+		(layer "B.Cu")
+		(net "/Row_3")
+	)
+	(segment
+		(start 233.7 81.4)
+		(end 236.25 78.85)
+		(width 0.25)
+		(layer "B.Cu")
+		(net "/Row_3")
+	)
+	(segment
 		(start 60.5725 125.215)
 		(end 61.7625 126.405)
@@
 	)
 	(segment
+		(start 232.0225 125.215)
+		(end 232.0225 122.35222)
+		(width 0.25)
+		(layer "B.Cu")
+		(net "/Row_3")
+	)
+	(segment
+		(start 251.325 47.275)
+		(end 251.35 47.25)
+		(width 0.25)
+		(layer "B.Cu")
+		(net "/Row_3")
+	)
+	(segment
 		(start 78.4325 126.405)
 		(end 79.6225 125.215)
@@
 	)
 	(segment
+		(start 237.25 99.8)
+		(end 235.45 98)
+		(width 0.25)
+		(layer "B.Cu")
+		(net "/Row_3")
+	)
+	(segment
 		(start 173.6825 126.405)
 		(end 157.0125 126.405)
@@
 	)
 	(segment
+		(start 251.35 47.25)
+		(end 250.7 46.6)
+		(width 0.25)
+		(layer "B.Cu")
+		(net "/Row_3")
+	)
+	(segment
+		(start 236.25 78.85)
+		(end 236.95 78.85)
+		(width 0.25)
+		(layer "B.Cu")
+		(net "/Row_3")
+	)
+	(segment
 		(start 272.50375 163.315)
 		(end 285.635 163.315)
 		(width 0.25)
 		(layer "B.Cu")
+		(net "/Row_3")
+	)
+	(segment
+		(start 250.7 46.6)
+		(end 248.05 46.6)
+		(width 0.25)
+		(layer "B.Cu")
