File: Computer Designs/CYKEYBOARD/CYKEYBOARD.kicad_pcb (KiCad board)
At the start: 2 copper layers, 528.3 x 165.1 mm, 344 parts, among them J1 Conn_01x12, J2 Conn_01x03, J3 Conn_01x03, K0 RESET, K13 READY, K14 ~~,,,,,,`, K15 !,,,,,,1, K16 @,,,,,,2, K17 #,,,,,,3, K18 $,,,,,,4, K19 %,,,,,,5, K20 ^,,,,,,6, K21 &,,,,,,7, K22 *,,,,,,8, K23 (,,,,,,9, K24 ),,,,,,0, K25 _,,,,,,-, K26 +,,,,,,=, K27 BACKSPACE, K28 HOME, K29 MON, K30 !,,,,,,1, K31 SAVE,,,,,,LOAD, K32 Q, K33 W, K34 E, K35 R, K36 T, K37 Y, K38 U, K39 I, K40 O, K41 P, K42 {,,,,,,[, K43 },,,,,,], K44 |,,,,,,\, K45 DEL, K46 BAS, K47 @,,,,,,2, K48 SHIFT,,,,,,LOCK, K49 A, K50 S, K51 D, K52 F, K53 G, K54 H, K55 J, K56 K, K57 L, K58 :,,,,,,;, K59 ",,,,,,', K60 ENTER, K61 SHIFT, K62 Z, K63 X, K64 C, K65 V, K66 B, K67 N, K68 M, K69 <,,,,,,,, K70 >,,,,,,., K71 ?,,,,,,/, K72 SHIFT, K73 ^, K74 CTRL, K75 CYKA,,,,,,TECH, K76 ALT, K77 Blank, K78 ALT, K79 FN, K80 SELECT, K81 CTRL, K82 <, K83 \/, K84 >, K85 #,,,,,,3, K86 $,,,,,,4, K87 BACKSPACE, K88 ),,,,,,0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

Commit message: Continued Compiler
Routing:
- net /PAUSE_LED: track 44.0 -> 446.8 mm, vias 2 -> 16
- net Net-(D3-A): track 0.00 -> 272.3 mm, vias 0 -> 17
- net /BIT0: track 0.00 -> 259.9 mm, vias 0 -> 14
- net /BIT1: track 0.00 -> 258.7 mm, vias 0 -> 10
- net Net-(U8A-C): track 59.0 -> 314.1 mm, vias 2 -> 25
- net /BUF-C0: track 99.5 -> 338.2 mm, vias 4 -> 14
- net Net-(U11-A7): track 0.00 -> 152.4 mm, vias 0 -> 9
- net /BUF-C14: track 76.3 -> 200.3 mm, vias 4 -> 15
- net /EO1: track 0.00 -> 121.4 mm, vias 0 -> 5
- net /BUF-C10: track 83.3 -> 203.9 mm, vias 5 -> 11
- net /BUF-C11: track 83.4 -> 201.8 mm, vias 4 -> 8
- net /BUF-C13: track 76.4 -> 194.6 mm, vias 4 -> 14
- net /BUF-C12: track 79.0 -> 191.6 mm, vias 2 -> 10
- net /GS1: track 0.00 -> 109.4 mm, vias 0 -> 9
- net /BUF-C2: track 80.9 -> 175.4 mm, vias 6 -> 13
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
Commit message: Continued
Parts:
- removed R138, R140: 2.2k, Resistor_THT:R_Axial_DIN0207_L6.3mm_D2.5mm_P10.16mm_Horizontal
Connections:
- U8 pad 1: Net-(U8A-C) -> /VCC
- U8 pad 10: Net-(U8B-~{R}) -> /VCC
- U8 pad 11: Net-(U8B-C) -> /VCC
- U8 pad 13: Net-(U8A-~{R}) -> /VCC
- U8 pad 4: Net-(U8A-C) -> /VCC
- U8 pad 8: Net-(U8B-C) -> /VCC
Routing:
- net /VCC: track 977.0 -> 1373.6 mm, vias 0 -> 29
- net Net-(U8B-~{R}): track 207.7 -> 0.00 mm, vias 15 -> 0
- net Net-(U8A-~{R}): track 194.8 -> 0.00 mm, vias 16 -> 0
- net Net-(U8A-C): track 314.1 -> 303.2 mm, vias 25 -> 22
- net Net-(U8B-C): track 247.3 -> 243.5 mm, vias 12 -> 14

Commit message: Continued
Routing:
- net Net-(U11-A3): track 0.00 -> 192.4 mm, vias 0 -> 15
- net /VCC: track 1373.6 -> 1186.1 mm, vias 29 -> 13
- net /GS2: track 21.3 -> 120.8 mm, vias 2 -> 9
- net Net-(U11-A4): track 0.00 -> 50.7 mm, vias 0 -> 4

Commit message: Continued
Routing:
- net Net-(U11-A5): track 0.00 -> 49.4 mm, vias 0 -> 4
Changed lines of the file:
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@@
+	)
+	(segment
+		(start 131.625 58.45)
+		(end 133.6 58.45)
+		(width 0.25)
+		(layer "F.Cu")
+		(net "Net-(U11-A5)")
+	)
+	(segment
+		(start 142.014009 63.635)
+		(end 150.99 63.635)
+		(width 0.25)
+		(layer "F.Cu")
+		(net "Net-(U11-A5)")
+	)
+	(segment
+		(start 133.6 58.45)
+		(end 133.75 58.6)
+		(width 0.25)
+		(layer "F.Cu")
+		(net "Net-(U11-A5)")
+	)
+	(segment
+		(start 140.075 61.695991)
+		(end 142.014009 63.635)
+		(width 0.25)
+		(layer "F.Cu")
+		(net "Net-(U11-A5)")
+	)
+	(segment
+		(start 140.075 60.875)
+		(end 140.075 61.695991)
+		(width 0.25)
+		(layer "F.Cu")
+		(net "Net-(U11-A5)")
+	)
+	(segment
+		(start 150.99 63.635)
+		(end 151.75 62.875)
+		(width 0.25)
+		(layer "F.Cu")
+		(net "Net-(U11-A5)")
+	)
+	(via
+		(at 151.75 62.875)
+		(size 0.25)
+		(drill 0.3)
+		(layers "F.Cu" "B.Cu")
+		(net "Net-(U11-A5)")
+	)
+	(via
+		(at 140.075 60.875)
+		(size 0.25)
+		(drill 0.3)
+		(layers "F.Cu" "B.Cu")
+		(net "Net-(U11-A5)")
+	)
+	(via
+		(at 133.75 58.6)
+		(size 0.25)
+		(drill 0.3)
+		(layers "F.Cu" "B.Cu")
+		(net "Net-(U11-A5)")
+	)
+	(via
+		(at 131.625 58.45)
+		(size 0.25)
+		(drill 0.3)
+		(layers "F.Cu" "B.Cu")
+		(net "Net-(U11-A5)")
+	)
+	(segment
+		(start 115.32 58.45)
+		(end 131.625 58.45)
+		(width 0.25)
+		(layer "B.Cu")
+		(net "Net-(U11-A5)")
+	)
+	(segment
+		(start 137.8 58.6)
+		(end 140.075 60.875)
+		(width 0.25)
+		(layer "B.Cu")
+		(net "Net-(U11-A5)")
+	)
+	(segment
+		(start 152.575 62.05)
+		(end 159.65 62.05)
+		(width 0.25)
+		(layer "B.Cu")
+		(net "Net-(U11-A5)")
+	)
+	(segment
+		(start 114.05 59.72)
+		(end 115.32 58.45)
+		(width 0.25)
+		(layer "B.Cu")
+		(net "Net-(U11-A5)")
+	)
+	(segment
+		(start 151.75 62.875)
+		(end 152.575 62.05)
+		(width 0.25)
+		(layer "B.Cu")
+		(net "Net-(U11-A5)")
+	)
+	(segment
+		(start 133.75 58.6)
+		(end 137.8 58.6)
+		(width 0.25)
+		(layer "B.Cu")
+		(net "Net-(U11-A5)")
 	)
 	(segment

Commit message: Continued
Routing:
- net Net-(U11-A4): track 50.7 -> 273.0 mm, vias 4 -> 21

Commit message: Continued
Routing:
- net Net-(U11-A5): track 49.4 -> 252.3 mm, vias 4 -> 21
