File: Computer Designs/6502-Cartridge-Design/6502-Cartridge-Design.kicad_sch (KiCad schematic)
At the start: 10 parts, among them J1 Conn_01x12_Pin, U1 74HC14, U2 23AA02M-IP, U3 7408, U4 AT25xxx, U5 MB85RS64

Commit message: Continued
Parts:
- U2: footprint Package_DIP:DIP-8_W7.62mm -> Package_SO:TSSOP-8_4.4x3mm_P0.65mm
Other:
- note added: "N01S830HAT22I RAM"
- note removed: "23A256 RAM"
Changed lines of the file:
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@@
 		)
 	)
-	(text "23A256\nRAM"
+	(text "N01S830HAT22I\nRAM"
 		(exclude_from_sim no)
 		(at 154.686 154.94 0)
@@
 			)
 		)
-		(property "Footprint" "Package_DIP:DIP-8_W7.62mm"
+		(property "Footprint" "Package_SO:TSSOP-8_4.4x3mm_P0.65mm"
 			(at 125.73 138.43 0)
 			(hide yes)

Commit message: Continued
Other:
- note added: "MB85RS64VYPNF-G-BCERE1 STORAGE"
- note removed: "FM25CL64B"
Changed lines of the file:
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@@
 		)
 	)
-	(text "FM25CL64B"
+	(text "MB85RS64VYPNF-G-BCERE1\nSTORAGE\n"
 		(exclude_from_sim no)
-		(at 232.41 139.192 0)
+		(at 240.538 139.192 0)
 		(effects
 			(font
