File: Computer Designs/6502-Cartridge-Design/6502-Cartridge-Design.kicad_pcb (KiCad board)
At the start: 2 copper layers, 76 x 60 mm, 14 parts, among them J1 Conn_01x12_Pin, U1 74HC14, U2 23AA02M-IP, U3 7408, U4 AT25xxx, U5 MB85RS64

Commit message: Continued
Routing:
- net Net-(J1-Pin_11): track 141.7 -> 143.0 mm
Changed lines of the file:
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@@
+	)
+	(segment
+		(start 117 65)
+		(end 115.6 63.6)
+		(width 0.3)
+		(layer "F.Cu")
+		(net "Net-(J1-Pin_11)")
 	)
 	(segment
@@
 	)
 	(segment
+		(start 124.7 70.5)
+		(end 119.2 65)
+		(width 0.3)
+		(layer "F.Cu")
+		(net "Net-(J1-Pin_11)")
+	)
+	(segment
 		(start 131.3 86)
 		(end 124.1 78.8)
@@
 	)
 	(segment
-		(start 124.7 70.5)
+		(start 115.6 63.6)
 		(end 115.6 61.4)
 		(width 0.3)
@@
 		(width 0.3)
 		(layer "F.Cu")
+		(net "Net-(J1-Pin_11)")
+	)
+	(segment
+		(start 119.2 65)
+		(end 117 65)
+		(width 0.3)
+		(layer "F.Cu")

Commit message: Continued
Parts:
- U2: footprint Package_DIP:DIP-8_W7.62mm -> Package_SO:TSSOP-8_4.4x3mm_P0.65mm
- moved U2 5.96 mm to (71.8, 73.9)
Routing:
- net Net-(J1-Pin_12): track 37.4 -> 73.6 mm
- net Net-(U2-~{CS}): track 47.1 -> 29.3 mm, vias 0 -> 1
- net Net-(J1-Pin_1): track 179.4 -> 162.0 mm
- net Net-(J1-Pin_10): track 120.9 -> 123.4 mm, vias 6 -> 7
- net Net-(J1-Pin_11): track 143.0 -> 145.2 mm
- net Net-(J1-Pin_9): track 149.8 -> 150.4 mm, vias 7 -> 5

Commit message: Continued
Other:
- board text added: "MB85RS64VYPNF-G-BCERE1 STOR"
- board text added: "N01S830HAT22I - RAM"
- board text removed: "23A256 RAM"
- board text removed: "FM25CL64B STOR"
Changed lines of the file:
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@@
 		(layer "Edge.Cuts")
 	)
-	(gr_text "23A256\nRAM"
-		(at 67.81 83.81 0)
+	(gr_text "N01S830HAT22I - RAM"
+		(at 65 70 0)
 		(layer "F.SilkS")
 		(effects
@@
 		)
 	)
-	(gr_text "FM25CL64B\nSTOR"
-		(at 128 95 0)
+	(gr_text "MB85RS64VYPNF-G-BCERE1\nSTOR"
+		(at 115.125 95.25 0)
 		(layer "F.SilkS")
 		(effects
